Commit message: gazebo and ros control interface

File: pa10_description/urdf/arm.transmission.xacro (robot description, xacro)
@@ -5,9 +5,11 @@
       <type>transmission_interface/SimpleTransmission</type>
       <actuator name="${name}_motor" >
+        <!--hardwareInterface>EffortJointInterface</hardwareInterface-->
+        <hardwareInterface>PositionJointInterface</hardwareInterface>
         <mechanicalReduction>${reduction}</mechanicalReduction>
       </actuator>
       <joint name="${name}">
-        <hardwareInterface>hardware_interface/PositionJointInterface</hardwareInterface>
-        <hardwareInterface>hardware_interface/EffortJointInterface</hardwareInterface>
+        <!--hardwareInterface>EffortJointInterface</hardwareInterface-->
+        <hardwareInterface>PositionJointInterface</hardwareInterface>
       </joint>
     </transmission>

File: pa10_description/urdf/pa10_csl.urdf.xacro (robot description, xacro)
@@ -5,15 +5,15 @@
 	<!-- NOT THE ACTUAL VALUE -->
 	<xacro:property name="arm_eps"            value="0.02" />
-	<xacro:property name="joint_1_max_effort" value="39.0"/>
-	<xacro:property name="joint_2_max_effort" value="39.0"/>
-	<xacro:property name="joint_3_max_effort" value="39.0"/>
-	<xacro:property name="joint_4_max_effort" value="39.0"/>
-	<xacro:property name="joint_5_max_effort" value="39.0"/>
-	<xacro:property name="joint_6_max_effort" value="39.0"/>
-	<xacro:property name="joint_7_max_effort" value="39.0"/>
+	<xacro:property name="joint_1_max_effort" value="150.0"/>
+	<xacro:property name="joint_2_max_effort" value="150.0"/>
+	<xacro:property name="joint_3_max_effort" value="150.0"/>
+	<xacro:property name="joint_4_max_effort" value="150.0"/>
+	<xacro:property name="joint_5_max_effort" value="150.0"/>
+	<xacro:property name="joint_6_max_effort" value="150.0"/>
+	<xacro:property name="joint_7_max_effort" value="150.0"/>
 	<!-- JOINTS POSITION LIMITS -->
 	<!-- Real Values: [177, 94, 174, 137, 255, 165, 255] (deg)-->
 	<xacro:property name="joint_1_max_position" value="${170.0 *pi/180.0}"/>
-	<xacro:property name="joint_2_max_position" value="${ 90.0 *pi/180.0}"/>
+	<xacro:property name="joint_2_max_position" value="${90.0 *pi/180.0}"/>
 	<xacro:property name="joint_3_max_position" value="${170.0 *pi/180.0}"/>
 	<xacro:property name="joint_4_max_position" value="${130.0 *pi/180.0}"/>
@@ -30,4 +30,22 @@
 	<xacro:property name="joint_6_max_velocity" value="${1.8*pi}"/>
 	<xacro:property name="joint_7_max_velocity" value="${1.8*pi}"/>
+    <!-- JOINT DYNAMICS DAMPING + FRICTION-->
+    <!-- >> !! Not Real Values !! << -->
+    <!-- DAMPING -->
+	<xacro:property name="joint_1_damping" value="0.01"/>
+	<xacro:property name="joint_2_damping" value="0.01"/>
+	<xacro:property name="joint_3_damping" value="0.01"/>
+	<xacro:property name="joint_4_damping" value="0.01"/>
+	<xacro:property name="joint_5_damping" value="0.01"/>
+	<xacro:property name="joint_6_damping" value="0.01"/>
+	<xacro:property name="joint_7_damping" value="0.01"/>
+	<!-- FRICTION -->
+	<xacro:property name="joint_1_friction" value="2.0"/>
+	<xacro:property name="joint_2_friction" value="2.0"/>
+	<xacro:property name="joint_3_friction" value="2.0"/>
+	<xacro:property name="joint_4_friction" value="2.0"/>
+	<xacro:property name="joint_5_friction" value="2.0"/>
+	<xacro:property name="joint_6_friction" value="2.0"/>
+	<xacro:property name="joint_7_friction" value="2.0"/>
 	<!-- Import all Gazebo-customization elements, including Gazebo colors -->
   <xacro:include filename="$(find pa10_description)/urdf/pa10csl.gazebo" />
@@ -56,5 +74,5 @@
     <inertial>
       <origin rpy="0 0 0" xyz="0 0 1"/>
-      <mass value="1"/>
+      <mass value="0.5"/>
       <inertia ixx="1" ixy="0.0" ixz="0.0" iyy="1" iyz="0.0" izz="1"/>
     </inertial>
@@ -79,5 +97,5 @@
     <inertial>
       <origin rpy="0 0 3.14" xyz="0 0 0"/>
-      <mass value="1"/>
+      <mass value="0.5"/>
       <inertia ixx="1" ixy="0.0" ixz="0.0" iyy="1" iyz="0.0" izz="1"/>
     </inertial>
@@ -101,5 +119,5 @@
     <inertial>
       <origin rpy="0 0 0" xyz="0 0 0.117"/>
-      <mass value="1"/>
+      <mass value="0.5"/>
       <inertia ixx="1" ixy="0.0" ixz="0.0" iyy="1" iyz="0.0" izz="1"/>
     </inertial>
@@ -123,5 +141,5 @@
     <inertial>
       <origin rpy="-1.57079 0 3.14159" xyz="0 0 0"/>
-      <mass value="1"/>
+      <mass value="0.5"/>
       <inertia ixx="1" ixy="0.0" ixz="0.0" iyy="1" iyz="0.0" izz="1"/>
     </inertial>
@@ -130,5 +148,5 @@
 		<inertial>
       <origin rpy="0 0 0" xyz="0 0 1"/>
-      <mass value="1"/>
+      <mass value="0.5"/>
       <inertia ixx="1" ixy="0.0" ixz="0.0" iyy="1" iyz="0.0" izz="1"/>
     </inertial>
@@ -152,5 +170,5 @@
     <inertial>
       <origin rpy="0 0 0" xyz="0 0.0 0.133"/>
-      <mass value="1"/>
+      <mass value="0.5"/>
       <inertia ixx="1" ixy="0.0" ixz="0.0" iyy="1" iyz="0.0" izz="1"/>
     </inertial>
@@ -174,5 +192,5 @@
     <inertial>
       <origin rpy="1.57079 0 0" xyz="0 0.003 0"/>
-      <mass value="1"/>
+      <mass value="0.5"/>
       <inertia ixx="1" ixy="0.0" ixz="0.0" iyy="1" iyz="0.0" izz="1"/>
     </inertial>
@@ -196,5 +214,5 @@
     <inertial>
       <origin rpy="0 0 0" xyz="0 0 0.195"/>
-      <mass value="1"/>
+      <mass value="0.5"/>
       <inertia ixx="1" ixy="0.0" ixz="0.0" iyy="1" iyz="0.0" izz="1"/>
     </inertial>
@@ -218,5 +236,5 @@
     <inertial>
       <origin rpy="1.57079 0 0" xyz="0 0 0"/>
-      <mass value="1"/>
+      <mass value="0.5"/>
       <inertia ixx="1" ixy="0.0" ixz="0.0" iyy="1" iyz="0.0" izz="1"/>
     </inertial>
@@ -249,5 +267,5 @@
     <inertial>
       <origin rpy="0 0 0" xyz="0 0 -0.045"/>
-      <mass value="0.5"/>
+      <mass value="0.001"/>
       <inertia ixx="1" ixy="0.0" ixz="0.0" iyy="1" iyz="0.0" izz="1"/>
     </inertial>
@@ -300,11 +318,13 @@
 	<!--   JOINTS    -->
   <!--************ -->
-	<joint name="fixed" type="fixed">
-    <origin rpy="${-pi/2.0} 0 0" xyz="0 0 1.35"/>
+  <joint name="fixed" type="fixed">
+    <!-- origin rpy="${-pi/2.0} 0 0" xyz="0 0 1.35"/ -->
+    <origin rpy="0 0 0" xyz="0 0 0.0"/>
     <parent link="world"/>
     <child link="base_link"/>
   </joint>
   <joint name="kinect" type="fixed">
-    <origin rpy="${-15.0*pi/180.0} 0 0" xyz="0.148 -0.48 -0.05"/>
+    <!-- origin rpy="${-15.0*pi/180.0} 0 0" xyz="0.148 -0.48 -0.05"/ -->
+    <origin rpy="${-125.0*pi/180.0} 0 ${pi}" xyz="0.148 0.48 1.8"/>
     <parent link="base_link"/>
     <child link="kinect2_rgb_optical_frame"/>
@@ -321,8 +341,9 @@
     <axis xyz="0 0 1"/>
     <limit effort="${joint_1_max_effort}" lower="${-joint_1_max_position}" upper="${joint_1_max_position}" velocity="${joint_1_max_velocity}"/>
-		<safety_controller k_position="20"
+    <safety_controller k_position="20"
                        k_velocity="20"
                        soft_lower_limit="${-joint_1_max_position + arm_eps}"
                        soft_upper_limit="${ joint_1_max_position - arm_eps}" />
+    <dynamics damping="${joint_1_damping}" friction="${joint_1_friction}" />
   </joint>
 	<joint name="S2" type="revolute">
@@ -336,4 +357,5 @@
                        soft_lower_limit="${-joint_2_max_position + arm_eps}"
                        soft_upper_limit="${ joint_2_max_position - arm_eps}" />
+    <dynamics damping="${joint_2_damping}" friction="${joint_2_friction}" />
   </joint>
 	<joint name="soldier_to_elbow_joint" type="fixed">
@@ -352,4 +374,5 @@
                        soft_lower_limit="${-joint_3_max_position + arm_eps}"
                        soft_upper_limit="${ joint_3_max_position - arm_eps}" />
+    <dynamics damping="${joint_3_damping}" friction="${joint_3_friction}" />
   </joint>
 	<joint name="E2" type="revolute">
@@ -363,4 +386,5 @@
                        soft_lower_limit="${-joint_4_max_position + arm_eps}"
                        soft_upper_limit="${ joint_4_max_position - arm_eps}" />
+    <dynamics damping="${joint_4_damping}" friction="${joint_4_friction}" />
   </joint>
 	<joint name="W1" type="revolute">
@@ -374,4 +398,5 @@
                        soft_lower_limit="${-joint_5_max_position + arm_eps}"
                        soft_upper_limit="${ joint_5_max_position - arm_eps}" />
+  <dynamics damping="${joint_5_damping}" friction="${joint_5_friction}" />
   </joint>
 	<joint name="W2" type="revolute">
@@ -385,4 +410,5 @@
                        soft_lower_limit="${-joint_6_max_position + arm_eps}"
                        soft_upper_limit="${ joint_6_max_position - arm_eps}" />
+    <dynamics damping="${joint_6_damping}" friction="${joint_6_friction}" />
   </joint>
 	<joint name="W3" type="revolute">
@@ -396,4 +422,5 @@
                        soft_lower_limit="${-joint_7_max_position + arm_eps}"
                        soft_upper_limit="${ joint_7_max_position - arm_eps}" />
+    <dynamics damping="${joint_7_damping}" friction="${joint_7_friction}" />
   </joint>
 	<!-- GRIPPER JOINTS -->
@@ -433,12 +460,12 @@
 	<!--    TRANSMITIONS     -->
 	<!-- ******************* -->
-	<xacro:arm_simple_transmission name="S1" reduction="1.0" />
-	<xacro:arm_simple_transmission name="S2" reduction="1.0" />
-	<xacro:arm_simple_transmission name="E1" reduction="1.0" />
-	<xacro:arm_simple_transmission name="E2" reduction="1.0" />
-	<xacro:arm_simple_transmission name="W1" reduction="1.0" />
-	<xacro:arm_simple_transmission name="W2" reduction="1.0" />
-	<xacro:arm_simple_transmission name="W3" reduction="1.0" />
-	<xacro:arm_simple_transmission name="finger_joint_1" reduction="1.0" />
-	<xacro:arm_simple_transmission name="finger_joint_2" reduction="1.0" />
+	<xacro:arm_simple_transmission name="S1" reduction="10" />
+	<xacro:arm_simple_transmission name="S2" reduction="10" />
+	<xacro:arm_simple_transmission name="E1" reduction="10" />
+	<xacro:arm_simple_transmission name="E2" reduction="10" />
+	<xacro:arm_simple_transmission name="W1" reduction="10" />
+	<xacro:arm_simple_transmission name="W2" reduction="10" />
+	<xacro:arm_simple_transmission name="W3" reduction="10" />
+	<xacro:arm_simple_transmission name="finger_joint_1" reduction="1" />
+	<xacro:arm_simple_transmission name="finger_joint_2" reduction="1" />
 </robot>

Commit message: minor changes

File: pa10_description/urdf/arm.transmission.xacro (robot description, xacro)
@@ -6,10 +6,10 @@
       <actuator name="${name}_motor" >
         <!--hardwareInterface>EffortJointInterface</hardwareInterface-->
-        <hardwareInterface>PositionJointInterface</hardwareInterface>
+        <hardwareInterface>VelocityJointInterface</hardwareInterface>
         <mechanicalReduction>${reduction}</mechanicalReduction>
       </actuator>
       <joint name="${name}">
         <!--hardwareInterface>EffortJointInterface</hardwareInterface-->
-        <hardwareInterface>PositionJointInterface</hardwareInterface>
+        <hardwareInterface>VelocityJointInterface</hardwareInterface>
       </joint>
     </transmission>

File: pa10_description/urdf/pa10_csl.urdf.xacro (robot description, xacro)
@@ -37,19 +37,19 @@
     <!-- >> !! Not Real Values !! << -->
     <!-- DAMPING -->
-	<xacro:property name="joint_1_damping" value="0.01"/>
-	<xacro:property name="joint_2_damping" value="0.01"/>
-	<xacro:property name="joint_3_damping" value="0.01"/>
-	<xacro:property name="joint_4_damping" value="0.01"/>
-	<xacro:property name="joint_5_damping" value="0.01"/>
-	<xacro:property name="joint_6_damping" value="0.01"/>
-	<xacro:property name="joint_7_damping" value="0.01"/>
+	<xacro:property name="joint_1_damping" value="0.1"/>
+	<xacro:property name="joint_2_damping" value="0.1"/>
+	<xacro:property name="joint_3_damping" value="0.1"/>
+	<xacro:property name="joint_4_damping" value="0.1"/>
+	<xacro:property name="joint_5_damping" value="0.1"/>
+	<xacro:property name="joint_6_damping" value="0.1"/>
+	<xacro:property name="joint_7_damping" value="0.1"/>
 	<!-- FRICTION -->
-	<xacro:property name="joint_1_friction" value="2.0"/>
-	<xacro:property name="joint_2_friction" value="2.0"/>
-	<xacro:property name="joint_3_friction" value="2.0"/>
-	<xacro:property name="joint_4_friction" value="2.0"/>
-	<xacro:property name="joint_5_friction" value="2.0"/>
-	<xacro:property name="joint_6_friction" value="2.0"/>
-	<xacro:property name="joint_7_friction" value="2.0"/>
+	<xacro:property name="joint_1_friction" value="0.7"/>
+	<xacro:property name="joint_2_friction" value="0.7"/>
+	<xacro:property name="joint_3_friction" value="0.7"/>
+	<xacro:property name="joint_4_friction" value="0.7"/>
+	<xacro:property name="joint_5_friction" value="0.7"/>
+	<xacro:property name="joint_6_friction" value="0.7"/>
+	<xacro:property name="joint_7_friction" value="0.7"/>
 	<!-- Import all Gazebo-customization elements, including Gazebo colors -->
   <xacro:include filename="$(find pa10_description)/urdf/pa10csl.gazebo.urdf.xacro" />

File: pa10_description/urdf/pa10csl.gazebo.urdf.xacro (robot description, xacro)
@@ -11,4 +11,6 @@
       </xacro:unless>
       <robotSimType>gazebo_ros_control/DefaultRobotHWSim</robotSimType>
+      <legacyModeNS>true</legacyModeNS>
+      <controlPeriod> 0.001</controlPeriod>
     </plugin>
   </gazebo>

Commit message: update moveit files

File: pa10_description/urdf/arm.transmission.xacro (robot description, xacro)
@@ -1,15 +1,29 @@
 <?xml version="1.0"?>
 <robot xmlns:xacro="http://ros.org/wiki/xacro">
-  <xacro:macro name="arm_simple_transmission" params="name reduction" >
+  <xacro:macro name="arm_simple_transmission" params="name reduction interface:=velocity" >
     <transmission name="${name}_trans">
       <type>transmission_interface/SimpleTransmission</type>
       <actuator name="${name}_motor" >
-        <!--hardwareInterface>EffortJointInterface</hardwareInterface-->
-        <hardwareInterface>VelocityJointInterface</hardwareInterface>
+        <xacro:if value="${interface == 'velocity'}">
+          <hardwareInterface>hardware_interface/VelocityJointInterface</hardwareInterface>
+        </xacro:if>
+        <xacro:if value="${interface == 'effort'}">
+          <hardwareInterface>hardware_interface/EffortJointInterface</hardwareInterface>
+        </xacro:if>
+        <xacro:if value="${interface == 'position'}">
+          <hardwareInterface>hardware_interface/PositionJointInterface</hardwareInterface>
+        </xacro:if>
         <mechanicalReduction>${reduction}</mechanicalReduction>
       </actuator>
       <joint name="${name}">
-        <!--hardwareInterface>EffortJointInterface</hardwareInterface-->
-        <hardwareInterface>VelocityJointInterface</hardwareInterface>
+        <xacro:if value="${interface == 'velocity'}">
+          <hardwareInterface>hardware_interface/VelocityJointInterface</hardwareInterface>
+        </xacro:if>
+        <xacro:if value="${interface == 'effort'}">
+          <hardwareInterface>hardware_interface/EffortJointInterface</hardwareInterface>
+        </xacro:if>
+        <xacro:if value="${interface == 'position'}">
+          <hardwareInterface>hardware_interface/PositionJointInterface</hardwareInterface>
+        </xacro:if>
       </joint>
     </transmission>

File: pa10_description/urdf/materials.xacro (robot description, xacro)
@@ -13,9 +13,12 @@
     <color rgba="0.2 0.2 0.2 1.0"/>
   </material>
-	 <material name="orange">
+  <material name="orange">
     <color rgba="${255/255} ${108/255} ${10/255} 1.0"/>
   </material>
   <material name="brown">
     <color rgba="${222/255} ${207/255} ${195/255} 1.0"/>
+  </material>
+  <material name="pa10_blue">
+    <color rgba="${140/255} ${217/255} ${227/255} 1.0"/>
   </material>
   <material name="red">

File: pa10_description/urdf/pa10_csl.urdf.xacro (robot description, xacro)
@@ -3,6 +3,8 @@
     <xacro:arg name="multiple" default="false"/> <!-- If multiple robots will be used -->
     <xacro:arg name="namespace" default=""/> <!-- namespace of the robot -->
+    <xacro:arg name="interface" default="velocity"/> <!-- namespace of the robot -->
     <xacro:property name="is_multiple" value="$(arg multiple)" />
     <xacro:property name="nsp" value="$(arg namespace)" />
+    <xacro:property name="HWInterface" value="$(arg interface)" />
 	<xacro:property name="pi" value="3.1415926535897931" />
 	<!-- JOINTS EFFORT LIMITS -->
@@ -37,19 +39,19 @@
     <!-- >> !! Not Real Values !! << -->
     <!-- DAMPING -->
-	<xacro:property name="joint_1_damping" value="0.1"/>
-	<xacro:property name="joint_2_damping" value="0.1"/>
-	<xacro:property name="joint_3_damping" value="0.1"/>
-	<xacro:property name="joint_4_damping" value="0.1"/>
-	<xacro:property name="joint_5_damping" value="0.1"/>
-	<xacro:property name="joint_6_damping" value="0.1"/>
-	<xacro:property name="joint_7_damping" value="0.1"/>
+	<xacro:property name="joint_1_damping" value="0.8"/>
+	<xacro:property name="joint_2_damping" value="0.8"/>
+	<xacro:property name="joint_3_damping" value="0.8"/>
+	<xacro:property name="joint_4_damping" value="0.8"/>
+	<xacro:property name="joint_5_damping" value="0.8"/>
+	<xacro:property name="joint_6_damping" value="0.8"/>
+	<xacro:property name="joint_7_damping" value="0.8"/>
 	<!-- FRICTION -->
-	<xacro:property name="joint_1_friction" value="0.7"/>
-	<xacro:property name="joint_2_friction" value="0.7"/>
-	<xacro:property name="joint_3_friction" value="0.7"/>
-	<xacro:property name="joint_4_friction" value="0.7"/>
-	<xacro:property name="joint_5_friction" value="0.7"/>
-	<xacro:property name="joint_6_friction" value="0.7"/>
-	<xacro:property name="joint_7_friction" value="0.7"/>
+	<xacro:property name="joint_1_friction" value="0.1"/>
+	<xacro:property name="joint_2_friction" value="0.1"/>
+	<xacro:property name="joint_3_friction" value="0.1"/>
+	<xacro:property name="joint_4_friction" value="0.1"/>
+	<xacro:property name="joint_5_friction" value="0.1"/>
+	<xacro:property name="joint_6_friction" value="0.1"/>
+	<xacro:property name="joint_7_friction" value="0.1"/>
 	<!-- Import all Gazebo-customization elements, including Gazebo colors -->
   <xacro:include filename="$(find pa10_description)/urdf/pa10csl.gazebo.urdf.xacro" />
@@ -89,6 +91,5 @@
         <mesh filename="package://pa10_description/pa10_stl/S1.stl" scale="1 1 1"/>
       </geometry>
-      <material name="">
-        <color rgba="0.34 0.35 0.36 1.0"/>
+      <material name="pa10_blue">
       </material>
     </visual>
@@ -112,5 +113,5 @@
       </geometry>
       <material name="">
-        <color rgba="0.33 0.96 0.53 1.5"/>
+        <color rgba="0.13 0.13 0.13 1.0"/>
       </material>
     </visual>
@@ -133,6 +134,5 @@
         <mesh filename="package://pa10_description/pa10_stl/S3.stl" scale="1 1 1"/>
       </geometry>
-      <material name="">
-        <color rgba="0.34 0.35 0.36 1.0"/>
+      <material name="pa10_blue">
       </material>
     </visual>
@@ -163,5 +163,5 @@
       </geometry>
       <material name="">
-        <color rgba="0.33 0.96 0.53 1.5"/>
+        <color rgba="0.13 0.13 0.13 1.5"/>
       </material>
     </visual>
@@ -207,5 +207,5 @@
       </geometry>
       <material name="">
-        <color rgba="0.33 0.96 0.53 1.5"/>
+        <color rgba="0.13 0.13 0.13 1.5"/>
       </material>
     </visual>
@@ -228,6 +228,5 @@
         <mesh filename="package://pa10_description/pa10_stl/W2.stl"  scale="1 1 1"/>
       </geometry>
-      <material name="">
-        <color rgba="0.34 0.35 0.36 1.0"/>
+      <material name="pa10_blue">
       </material>
     </visual>
@@ -328,6 +327,6 @@
     <child link="base_link"/>
   </joint>
+  <!--
   <joint name="kinect" type="fixed">
-    <!-- origin rpy="${-15.0*pi/180.0} 0 0" xyz="0.148 -0.48 -0.05"/ -->
     <origin rpy="${-125.0*pi/180.0} 0 ${pi}" xyz="0.148 0.48 1.8"/>
     <parent link="base_link"/>
@@ -339,4 +338,5 @@
     <child link="kinect2_ir_optical_frame"/>
   </joint>
+ -->
 	<joint name="S1" type="revolute">
     <origin rpy="0 0 0" xyz="0 0 0.2"/>
@@ -464,12 +464,12 @@
 	<!--    TRANSMITIONS     -->
 	<!-- ******************* -->
-	<xacro:arm_simple_transmission name="S1" reduction="10" />
-	<xacro:arm_simple_transmission name="S2" reduction="10" />
-	<xacro:arm_simple_transmission name="E1" reduction="10" />
-	<xacro:arm_simple_transmission name="E2" reduction="10" />
-	<xacro:arm_simple_transmission name="W1" reduction="10" />
-	<xacro:arm_simple_transmission name="W2" reduction="10" />
-	<xacro:arm_simple_transmission name="W3" reduction="10" />
-	<xacro:arm_simple_transmission name="finger_joint_1" reduction="1" />
-	<xacro:arm_simple_transmission name="finger_joint_2" reduction="1" />
+	<xacro:arm_simple_transmission name="S1" reduction="10" interface="${HWInterface}" />
+	<xacro:arm_simple_transmission name="S2" reduction="10" interface="${HWInterface}"/>
+	<xacro:arm_simple_transmission name="E1" reduction="10" interface="${HWInterface}"/>
+	<xacro:arm_simple_transmission name="E2" reduction="10" interface="${HWInterface}"/>
+	<xacro:arm_simple_transmission name="W1" reduction="10" interface="${HWInterface}"/>
+	<xacro:arm_simple_transmission name="W2" reduction="10" interface="${HWInterface}"/>
+	<xacro:arm_simple_transmission name="W3" reduction="10" interface="${HWInterface}"/>
+	<xacro:arm_simple_transmission name="finger_joint_1" reduction="1" interface="velocity"/>
+	<xacro:arm_simple_transmission name="finger_joint_2" reduction="1" interface="velocity"/>
 </robot>

File: pa10_description/urdf/pa10csl.gazebo.urdf.xacro (robot description, xacro)
@@ -19,5 +19,7 @@
     <mu1>0.5</mu1>
     <mu2>0.5</mu2>
-    <material>Gazebo/Grey</material>
+    <material name="pa10_blue">
+      Gazebo/Grey
+    </material>
   </gazebo>
   <!-- Link1 -->
@@ -29,5 +31,7 @@
     <mu1>0.5</mu1>
     <mu2>0.5</mu2>
-    <material>Gazebo/Grey</material>
+    <material name="pa10_blue">
+      Gazebo/Grey
+    </material>
   </gazebo>
   <!-- Link3 -->
@@ -41,5 +45,7 @@
     <mu1>0.5</mu1>
     <mu2>0.5</mu2>
-    <material>Gazebo/Grey</material>
+    <material name="pa10_blue">
+      Gazebo/Grey
+    </material>
   </gazebo>
   <!-- Link5 -->
@@ -53,10 +59,14 @@
     <mu1>0.5</mu1>
     <mu2>0.5</mu2>
-    <material>Gazebo/Grey</material>
+    <material name="pa10_blue">
+      Gazebo/Grey
+    </material>
   </gazebo>
 	<gazebo reference="link_wrist_2">
     <mu1>0.5</mu1>
     <mu2>0.5</mu2>
-    <material>Gazebo/Grey</material>
+    <material>
+      Gazebo/Blue
+    </material>
   </gazebo>
 	<gazebo reference="link_gripper_base">
