Commit message: change colors

File: pa10_description/urdf/pa10csl.gazebo.urdf.xacro (robot description, xacro)
@@ -5,8 +5,8 @@
     <plugin name="gazebo_ros_control" filename="libgazebo_ros_control.so">
       <xacro:if value="${is_multiple}">
-          <robotNamespace>/${nsp}</robotNamespace>
+        <robotNamespace>/${nsp}</robotNamespace>
       </xacro:if>
       <xacro:unless value="${is_multiple}">
-          <robotNamespace></robotNamespace>
+        <robotNamespace></robotNamespace>
       </xacro:unless>
       <robotSimType>gazebo_ros_control/DefaultRobotHWSim</robotSimType>
@@ -15,15 +15,25 @@
     </plugin>
   </gazebo>
-<!-- base_link -->
+  <!-- base_link -->
   <gazebo reference="base_link">
     <mu1>0.5</mu1>
     <mu2>0.5</mu2>
-    <material name="pa10_blue">
-      Gazebo/Grey
-    </material>
+    <visual>
+      <material>
+        <ambient>0.55 0.85 0.89 1.0</ambient>
+        <diffuse>.7 .7 .7  1.0</diffuse>
+        <specular>0.01 0.01 0.01 1.000000 1.500000</specular>
+      </material>
+    </visual>
   </gazebo>
   <!-- Link1 -->
   <gazebo reference="link_shoulder_1">
-    <material>Gazebo/Blue</material>
+    <visual>
+      <material>
+        <ambient>0.88 0.88 0.88 1.0</ambient>
+        <diffuse>.7 .7 .7  1.0</diffuse>
+        <specular>0.01 0.01 0.01 1.000000 1.500000</specular>
+      </material>
+    </visual>
   </gazebo>
   <!-- Link2 -->
@@ -31,7 +41,11 @@
     <mu1>0.5</mu1>
     <mu2>0.5</mu2>
-    <material name="pa10_blue">
-      Gazebo/Grey
-    </material>
+    <visual>
+      <material>
+        <ambient>0.55 0.85 0.89 1.0</ambient>
+        <diffuse>.7 .7 .7  1.0</diffuse>
+        <specular>0.01 0.01 0.01 1.000000 1.500000</specular>
+      </material>
+    </visual>
   </gazebo>
   <!-- Link3 -->
@@ -39,5 +53,11 @@
     <mu1>0.5</mu1>
     <mu2>0.5</mu2>
-    <material>Gazebo/Blue</material>
+    <visual>
+      <material>
+        <ambient>0.88 0.88 0.88 1.0</ambient>
+        <diffuse>.7 .7 .7  1.0</diffuse>
+        <specular>0.01 0.01 0.01 1.000000 1.500000</specular>
+      </material>
+    </visual>
   </gazebo>
   <!-- Link4 -->
@@ -45,7 +65,11 @@
     <mu1>0.5</mu1>
     <mu2>0.5</mu2>
-    <material name="pa10_blue">
-      Gazebo/Grey
-    </material>
+    <visual>
+      <material>
+        <ambient>0.55 0.85 0.89 1.0</ambient>
+        <diffuse>.7 .7 .7  1.0</diffuse>
+        <specular>0.01 0.01 0.01 1.000000 1.500000</specular>
+      </material>
+    </visual>
   </gazebo>
   <!-- Link5 -->
@@ -53,5 +77,11 @@
     <mu1>0.5</mu1>
     <mu2>0.5</mu2>
-    <material>Gazebo/Blue</material>
+    <visual>
+      <material>
+        <ambient>0.88 0.88 0.88 1.0</ambient>
+        <diffuse>.7 .7 .7  1.0</diffuse>
+        <specular>0.01 0.01 0.01 1.000000 1.500000</specular>
+      </material>
+    </visual>
   </gazebo>
   <!-- Link6 -->
@@ -59,26 +89,34 @@
     <mu1>0.5</mu1>
     <mu2>0.5</mu2>
-    <material name="pa10_blue">
-      Gazebo/Grey
-    </material>
+    <visual>
+      <material>
+        <ambient>0.55 0.85 0.89 1.0</ambient>
+        <diffuse>.7 .7 .7  1.0</diffuse>
+        <specular>0.01 0.01 0.01 1.000000 1.500000</specular>
+      </material>
+    </visual>
   </gazebo>
-	<gazebo reference="link_wrist_2">
+  <gazebo reference="link_wrist_3">
     <mu1>0.5</mu1>
     <mu2>0.5</mu2>
-    <material>
-      Gazebo/Blue
-    </material>
+    <visual>
+      <material>
+        <ambient>0.55 0.85 0.89 1.0</ambient>
+        <diffuse>.7 .7 .7  1.0</diffuse>
+        <specular>0.01 0.01 0.01 1.000000 1.500000</specular>
+      </material>
+    </visual>
   </gazebo>
-	<gazebo reference="link_gripper_base">
+  <gazebo reference="link_gripper_base">
     <mu1>0.5</mu1>
     <mu2>0.5</mu2>
     <material>Gazebo/Grey</material>
   </gazebo>
-	<gazebo reference="link_finger_1">
+  <gazebo reference="link_finger_1">
     <mu1>1000.5</mu1>
     <mu2>1000.5</mu2>
     <material>Gazebo/Orange</material>
   </gazebo>
-	<gazebo reference="link_finger_2">
+  <gazebo reference="link_finger_2">
     <mu1>1000.5</mu1>
     <mu2>1000.5</mu2>
