Commit message: pa10 multi robots

File: pa10_description/urdf/pa10_csl.urdf.xacro (robot description, xacro)
@@ -1,4 +1,8 @@
 <?xml version="1.0" ?>
 <robot name="pa10"  xmlns:xacro="http://www.ros.org/wiki/xacro">
+    <xacro:arg name="multiple" default="false"/> <!-- If multiple robots will be used -->
+    <xacro:arg name="namespace" default=""/> <!-- namespace of the robot -->
+    <xacro:property name="is_multiple" value="$(arg multiple)" />
+    <xacro:property name="nsp" value="$(arg namespace)" />
 	<xacro:property name="pi" value="3.1415926535897931" />
 	<!-- JOINTS EFFORT LIMITS -->
@@ -49,5 +53,5 @@
 	<xacro:property name="joint_7_friction" value="2.0"/>
 	<!-- Import all Gazebo-customization elements, including Gazebo colors -->
-  <xacro:include filename="$(find pa10_description)/urdf/pa10csl.gazebo" />
+  <xacro:include filename="$(find pa10_description)/urdf/pa10csl.gazebo.urdf.xacro" />
 	<!-- Import Rviz colors -->
   <xacro:include filename="$(find pa10_description)/urdf/materials.xacro" />

Commit message: minor modifications in urdf

File: pa10_description/urdf/pa10_csl.urdf.xacro (robot description, xacro)
@@ -113,5 +113,5 @@
       </geometry>
       <material name="">
-        <color rgba="0.13 0.13 0.13 1.0"/>
+        <color rgba="0.88 0.88 0.88 1.0"/>
       </material>
     </visual>
@@ -151,5 +151,5 @@
 	<link name="link_shoulder_to_elbow">
 		<inertial>
-      <origin rpy="0 0 0" xyz="0 0 1"/>
+      <origin rpy="0 0 0" xyz="0 0 0"/>
       <mass value="0.5"/>
       <inertia ixx="1" ixy="0.0" ixz="0.0" iyy="1" iyz="0.0" izz="1"/>
@@ -163,5 +163,5 @@
       </geometry>
       <material name="">
-        <color rgba="0.13 0.13 0.13 1.5"/>
+        <color rgba="0.88 0.88 0.88 1.0"/>
       </material>
     </visual>
@@ -184,6 +184,5 @@
         <mesh filename="package://pa10_description/pa10_stl/E2.stl" scale="1 1 1"/>
       </geometry>
-      <material name="">
-        <color rgba="0.34 0.35 0.36 1.0"/>
+      <material name="pa10_blue">
       </material>
     </visual>
@@ -207,5 +206,5 @@
       </geometry>
       <material name="">
-        <color rgba="0.13 0.13 0.13 1.5"/>
+        <color rgba="0.88 0.88 0.88 1.0"/>
       </material>
     </visual>
@@ -327,5 +326,4 @@
     <child link="base_link"/>
   </joint>
-  <!--
   <joint name="kinect" type="fixed">
     <origin rpy="${-125.0*pi/180.0} 0 ${pi}" xyz="0.148 0.48 1.8"/>
@@ -338,5 +336,4 @@
     <child link="kinect2_ir_optical_frame"/>
   </joint>
- -->
 	<joint name="S1" type="revolute">
     <origin rpy="0 0 0" xyz="0 0 0.2"/>

Commit message: update inertia

File: pa10_description/urdf/pa10_csl.urdf.xacro (robot description, xacro)
@@ -1,91 +1,101 @@
 <?xml version="1.0" ?>
-<robot name="pa10"  xmlns:xacro="http://www.ros.org/wiki/xacro">
-    <xacro:arg name="multiple" default="false"/> <!-- If multiple robots will be used -->
-    <xacro:arg name="namespace" default=""/> <!-- namespace of the robot -->
-    <xacro:arg name="interface" default="velocity"/> <!-- namespace of the robot -->
-    <xacro:property name="is_multiple" value="$(arg multiple)" />
-    <xacro:property name="nsp" value="$(arg namespace)" />
-    <xacro:property name="HWInterface" value="$(arg interface)" />
-	<xacro:property name="pi" value="3.1415926535897931" />
-	<!-- JOINTS EFFORT LIMITS -->
-	<!-- NOT THE ACTUAL VALUE -->
-	<xacro:property name="arm_eps"            value="0.02" />
-	<xacro:property name="joint_1_max_effort" value="150.0"/>
-	<xacro:property name="joint_2_max_effort" value="150.0"/>
-	<xacro:property name="joint_3_max_effort" value="150.0"/>
-	<xacro:property name="joint_4_max_effort" value="150.0"/>
-	<xacro:property name="joint_5_max_effort" value="150.0"/>
-	<xacro:property name="joint_6_max_effort" value="150.0"/>
-	<xacro:property name="joint_7_max_effort" value="150.0"/>
-	<!-- JOINTS POSITION LIMITS -->
-	<!-- Real Values: [177, 94, 174, 137, 255, 165, 255] (deg)-->
-	<xacro:property name="joint_1_max_position" value="${170.0 *pi/180.0}"/>
-	<xacro:property name="joint_2_max_position" value="${90.0 *pi/180.0}"/>
-	<xacro:property name="joint_3_max_position" value="${170.0 *pi/180.0}"/>
-	<xacro:property name="joint_4_max_position" value="${130.0 *pi/180.0}"/>
-	<xacro:property name="joint_5_max_position" value="${250.0 *pi/180.0}"/>
-	<xacro:property name="joint_6_max_position" value="${160.0 *pi/180.0}"/>
-	<xacro:property name="joint_7_max_position" value="${250.0 *pi/180.0}"/>
-	<!-- JOINTS VELOCITIE LIMITS-->
-	<!-- Real Values: [1, 1, 2, 2, 2, 2*pi, 2*pi] (rad/sec)-->
-	<xacro:property name="joint_1_max_velocity" value="0.85"/>
-	<xacro:property name="joint_2_max_velocity" value="0.85"/>
-	<xacro:property name="joint_3_max_velocity" value="1.85"/>
-	<xacro:property name="joint_4_max_velocity" value="1.85"/>
-	<xacro:property name="joint_5_max_velocity" value="1.85"/>
-	<xacro:property name="joint_6_max_velocity" value="${1.8*pi}"/>
-	<xacro:property name="joint_7_max_velocity" value="${1.8*pi}"/>
-    <!-- JOINT DYNAMICS DAMPING + FRICTION-->
-    <!-- >> !! Not Real Values !! << -->
-    <!-- DAMPING -->
-	<xacro:property name="joint_1_damping" value="0.8"/>
-	<xacro:property name="joint_2_damping" value="0.8"/>
-	<xacro:property name="joint_3_damping" value="0.8"/>
-	<xacro:property name="joint_4_damping" value="0.8"/>
-	<xacro:property name="joint_5_damping" value="0.8"/>
-	<xacro:property name="joint_6_damping" value="0.8"/>
-	<xacro:property name="joint_7_damping" value="0.8"/>
-	<!-- FRICTION -->
-	<xacro:property name="joint_1_friction" value="0.1"/>
-	<xacro:property name="joint_2_friction" value="0.1"/>
-	<xacro:property name="joint_3_friction" value="0.1"/>
-	<xacro:property name="joint_4_friction" value="0.1"/>
-	<xacro:property name="joint_5_friction" value="0.1"/>
-	<xacro:property name="joint_6_friction" value="0.1"/>
-	<xacro:property name="joint_7_friction" value="0.1"/>
-	<!-- Import all Gazebo-customization elements, including Gazebo colors -->
+<robot name="pa10"
+  xmlns:xacro="http://www.ros.org/wiki/xacro">
+  <xacro:arg name="multiple" default="false"/>
+  <!-- If multiple robots will be used -->
+  <xacro:arg name="namespace" default=""/>
+  <!-- namespace of the robot -->
+  <xacro:arg name="interface" default="velocity"/>
+  <!-- namespace of the robot -->
+  <xacro:arg name="enable_camera" default="false"/>
+  <xacro:property name="is_multiple" value="$(arg multiple)" />
+  <xacro:property name="nsp" value="$(arg namespace)" />
+  <xacro:property name="HWInterface" value="$(arg interface)" />
+  <xacro:property name="enable_camera_" value="$(arg enable_camera)" />
+  <xacro:property name="pi" value="3.1415926535897931" />
+  <!-- JOINTS EFFORT LIMITS -->
+  <!-- NOT THE ACTUAL VALUE -->
+  <xacro:property name="arm_eps" value="0.02" />
+  <xacro:property name="joint_1_max_effort" value="150.0"/>
+  <xacro:property name="joint_2_max_effort" value="150.0"/>
+  <xacro:property name="joint_3_max_effort" value="150.0"/>
+  <xacro:property name="joint_4_max_effort" value="150.0"/>
+  <xacro:property name="joint_5_max_effort" value="150.0"/>
+  <xacro:property name="joint_6_max_effort" value="150.0"/>
+  <xacro:property name="joint_7_max_effort" value="150.0"/>
+  <!-- JOINTS POSITION LIMITS -->
+  <!-- Real Values: [177, 94, 174, 137, 255, 165, 255] (deg)-->
+  <xacro:property name="joint_1_max_position" value="${170.0 *pi/180.0}"/>
+  <xacro:property name="joint_2_max_position" value="${90.0 *pi/180.0}"/>
+  <xacro:property name="joint_3_max_position" value="${170.0 *pi/180.0}"/>
+  <xacro:property name="joint_4_max_position" value="${130.0 *pi/180.0}"/>
+  <xacro:property name="joint_5_max_position" value="${250.0 *pi/180.0}"/>
+  <xacro:property name="joint_6_max_position" value="${160.0 *pi/180.0}"/>
+  <xacro:property name="joint_7_max_position" value="${250.0 *pi/180.0}"/>
+  <!-- JOINTS VELOCITIE LIMITS-->
+  <!-- Real Values: [1, 1, 2, 2, 2, 2*pi, 2*pi] (rad/sec)-->
+  <xacro:property name="joint_1_max_velocity" value="0.85"/>
+  <xacro:property name="joint_2_max_velocity" value="0.85"/>
+  <xacro:property name="joint_3_max_velocity" value="1.85"/>
+  <xacro:property name="joint_4_max_velocity" value="1.85"/>
+  <xacro:property name="joint_5_max_velocity" value="1.85"/>
+  <xacro:property name="joint_6_max_velocity" value="${1.8*pi}"/>
+  <xacro:property name="joint_7_max_velocity" value="${1.8*pi}"/>
+  <!-- JOINT DYNAMICS DAMPING + FRICTION-->
+  <!-- >> !! Not Real Values !! << -->
+  <!-- DAMPING -->
+  <xacro:property name="joint_1_damping" value="0.8"/>
+  <xacro:property name="joint_2_damping" value="0.8"/>
+  <xacro:property name="joint_3_damping" value="0.8"/>
+  <xacro:property name="joint_4_damping" value="0.8"/>
+  <xacro:property name="joint_5_damping" value="0.8"/>
+  <xacro:property name="joint_6_damping" value="0.8"/>
+  <xacro:property name="joint_7_damping" value="0.8"/>
+  <xacro:property name="joint_finger_damping" value="0.8"/>
+  <!-- FRICTION -->
+  <xacro:property name="joint_1_friction" value="0.1"/>
+  <xacro:property name="joint_2_friction" value="0.1"/>
+  <xacro:property name="joint_3_friction" value="0.1"/>
+  <xacro:property name="joint_4_friction" value="0.1"/>
+  <xacro:property name="joint_5_friction" value="0.1"/>
+  <xacro:property name="joint_6_friction" value="0.1"/>
+  <xacro:property name="joint_7_friction" value="0.1"/>
+  <xacro:property name="joint_finger_friction" value="0.1"/>
+  <!-- Import all Gazebo-customization elements, including Gazebo colors -->
   <xacro:include filename="$(find pa10_description)/urdf/pa10csl.gazebo.urdf.xacro" />
-	<!-- Import Rviz colors -->
+  <!-- Import Rviz colors -->
   <xacro:include filename="$(find pa10_description)/urdf/materials.xacro" />
-	<!-- Import Transmitions -->
-	<xacro:include filename="$(find pa10_description)/urdf/arm.transmission.xacro"/>
-	<!-- LINKS -->
-	<link name="world"/>
-	<link name="kinect2_rgb_optical_frame">
-		<visual>
-			<origin rpy="${pi} ${-pi/2.0} ${-pi/2.0}" xyz="0 0 0"/>
-      <geometry>
-        <mesh filename="package://pa10_description/sensors_3D_models/kinect.dae" scale="1 1 1"/>
-      </geometry>
-      <material name="">
-        <color rgba="0.0 0.0 0.0 1.0"/>
-      </material>
-    </visual>
-		<collision>
-      <origin rpy="${pi} ${-pi/2.0} ${-pi/2.0}" xyz="0 0 0"/>
-      <geometry>
-        <mesh filename="package://pa10_description/sensors_3D_models/kinect.dae" scale="1 1 1"/>
-      </geometry>
-    </collision>
-    <inertial>
-      <origin rpy="0 0 0" xyz="0 0 1"/>
-      <mass value="0.5"/>
-      <inertia ixx="1" ixy="0.0" ixz="0.0" iyy="1" iyz="0.0" izz="1"/>
-    </inertial>
-  </link>
-	<link name="kinect2_ir_optical_frame"/>
-	<link name="base_link">
-		<visual>
-			<origin rpy="0 0 3.14" xyz="0 0 0"/>
+  <!-- Import Transmitions -->
+  <xacro:include filename="$(find pa10_description)/urdf/arm.transmission.xacro"/>
+  <!-- LINKS -->
+  <link name="world"/>
+  <xacro:if value="${enable_camera_}">
+    <link name="kinect2_rgb_optical_frame">
+      <visual>
+        <origin rpy="${pi} ${-pi/2.0} ${-pi/2.0}" xyz="0 0 0"/>
+        <geometry>
+          <mesh filename="package://pa10_description/sensors_3D_models/kinect.dae" scale="1 1 1"/>
+        </geometry>
+        <material name="">
+          <color rgba="0.0 0.0 0.0 1.0"/>
+        </material>
+      </visual>
+      <collision>
+        <origin rpy="${pi} ${-pi/2.0} ${-pi/2.0}" xyz="0 0 0"/>
+        <geometry>
+          <mesh filename="package://pa10_description/sensors_3D_models/kinect.dae" scale="1 1 1"/>
+        </geometry>
+      </collision>
+      <inertial>
+        <origin rpy="0 0 0" xyz="0 0 1"/>
+        <mass value="0.5"/>
+        <inertia ixx="0.001" ixy="0.0" ixz="0.0" iyy="0.001" iyz="0.0" izz="0.001"/>
+      </inertial>
+    </link>
+    <link name="kinect2_ir_optical_frame"/>
+  </xacro:if>
+  <link name="base_link">
+    <visual>
+      <origin rpy="0 0 3.14" xyz="0 0 0"/>
       <geometry>
         <mesh filename="package://pa10_description/pa10_stl/S1.stl" scale="1 1 1"/>
@@ -94,5 +104,5 @@
       </material>
     </visual>
-		<collision>
+    <collision>
       <origin rpy="0 0 3.14" xyz="0 0 0"/>
       <geometry>
@@ -101,10 +111,10 @@
     </collision>
     <inertial>
-      <origin rpy="0 0 3.14" xyz="0 0 0"/>
-      <mass value="0.5"/>
-      <inertia ixx="1" ixy="0.0" ixz="0.0" iyy="1" iyz="0.0" izz="1"/>
-    </inertial>
-  </link>
-	<link name="link_shoulder_1">
+      <origin rpy="0 0 3.14" xyz="0 0 0.1"/>
+      <mass value="0.5"/>
+      <xacro:inertia_cylinder height="0.2"  radius = "0.1" mass="0.5"/>
+    </inertial>
+  </link>
+  <link name="link_shoulder_1">
     <visual>
       <origin rpy="0 0 0" xyz="0 0 0.117"/>
@@ -116,5 +126,5 @@
       </material>
     </visual>
-		<collision>
+    <collision>
       <origin rpy="0 0 0" xyz="0 0 0.117"/>
       <geometry>
@@ -125,8 +135,8 @@
       <origin rpy="0 0 0" xyz="0 0 0.117"/>
       <mass value="0.5"/>
-      <inertia ixx="1" ixy="0.0" ixz="0.0" iyy="1" iyz="0.0" izz="1"/>
-    </inertial>
-	</link>
-	<link name="link_shoulder_2">
+      <xacro:inertia_cylinder height="0.12"  radius = "0.08" mass="0.5"/>
+    </inertial>
+  </link>
+  <link name="link_shoulder_2">
     <visual>
       <origin rpy="-1.57079 0 3.14159" xyz="0 0 0"/>
@@ -144,17 +154,17 @@
     </collision>
     <inertial>
-      <origin rpy="-1.57079 0 3.14159" xyz="0 0 0"/>
-      <mass value="0.5"/>
-      <inertia ixx="1" ixy="0.0" ixz="0.0" iyy="1" iyz="0.0" izz="1"/>
-    </inertial>
-  </link>
-	<link name="link_shoulder_to_elbow">
-		<inertial>
-      <origin rpy="0 0 0" xyz="0 0 0"/>
-      <mass value="0.5"/>
-      <inertia ixx="1" ixy="0.0" ixz="0.0" iyy="1" iyz="0.0" izz="1"/>
-    </inertial>
-	</link>
-	<link name="link_elbow_1">
+      <origin rpy="-1.57079 0 3.14159" xyz="0 -0.22 0.0"/>
+      <mass value="0.5"/>
+      <xacro:inertia_cylinder height="0.18"  radius = "0.05" mass="0.5" axis="0"/>
+    </inertial>
+  </link>
+  <link name="link_shoulder_to_elbow">
+    <inertial>
+      <origin rpy="0 0 0" xyz="0 0 0.22"/>
+      <mass value="0.5"/>
+      <inertia ixx="0.001" ixy="0.0" ixz="0.0" iyy="0.001" iyz="0.0" izz="0.001"/>
+    </inertial>
+  </link>
+  <link name="link_elbow_1">
     <visual>
       <origin rpy="0 0 0" xyz="0 0.0 0.133"/>
@@ -175,5 +185,5 @@
       <origin rpy="0 0 0" xyz="0 0.0 0.133"/>
       <mass value="0.5"/>
-      <inertia ixx="1" ixy="0.0" ixz="0.0" iyy="1" iyz="0.0" izz="1"/>
+      <xacro:inertia_cylinder height="0.12"  radius = "0.08" mass="0.5"/>
     </inertial>
   </link>
@@ -188,5 +198,5 @@
     </visual>
     <collision>
-      <origin rpy="-1.57079 0 0" xyz="0 0.003 0"/>
+      <origin rpy="1.57079 0 0" xyz="0 0.003 0"/>
       <geometry>
         <mesh filename="package://pa10_description/pa10_stl_collision/E2_collision.stl" scale="1 1 1"/>
@@ -194,10 +204,10 @@
     </collision>
     <inertial>
-      <origin rpy="1.57079 0 0" xyz="0 0.003 0"/>
-      <mass value="0.5"/>
-      <inertia ixx="1" ixy="0.0" ixz="0.0" iyy="1" iyz="0.0" izz="1"/>
-    </inertial>
-  </link>
-	<link name="link_wrist_1">
+      <origin rpy="1.57079 0 0" xyz="0 -0.15 0"/>
+      <mass value="0.5"/>
+      <xacro:inertia_cylinder height="0.15"  radius = "0.05" mass="0.5" axis="0"/>
+    </inertial>
+  </link>
+  <link name="link_wrist_1">
     <visual>
       <origin rpy="0 0 0" xyz="0 0 0.195"/>
@@ -218,12 +228,12 @@
       <origin rpy="0 0 0" xyz="0 0 0.195"/>
       <mass value="0.5"/>
-      <inertia ixx="1" ixy="0.0" ixz="0.0" iyy="1" iyz="0.0" izz="1"/>
-    </inertial>
-  </link>
-	<link name="link_wrist_2">
+      <xacro:inertia_cylinder height="0.15"  radius = "0.08" mass="0.5"/>
+    </inertial>
+  </link>
+  <link name="link_wrist_2">
     <visual>
       <origin rpy="1.57079 0 0" xyz="0 0 0"/>
       <geometry>
-        <mesh filename="package://pa10_description/pa10_stl/W2.stl"  scale="1 1 1"/>
+        <mesh filename="package://pa10_description/pa10_stl/W2.stl" scale="1 1 1"/>
       </geometry>
       <material name="pa10_blue">
@@ -233,5 +243,5 @@
       <origin rpy="1.57079 0 0" xyz="0 0 0"/>
       <geometry>
-        <mesh filename="package://pa10_description/pa10_stl_collision/W2_collision.stl"  scale="1 1 1"/>
+        <mesh filename="package://pa10_description/pa10_stl_collision/W2_collision.stl" scale="1 1 1"/>
       </geometry>
     </collision>
@@ -239,65 +249,64 @@
       <origin rpy="1.57079 0 0" xyz="0 0 0"/>
       <mass value="0.5"/>
-      <inertia ixx="1" ixy="0.0" ixz="0.0" iyy="1" iyz="0.0" izz="1"/>
-    </inertial>
-  </link>
-	<link name="link_wrist_3"/>
-	<link name="link_ee_tool">
-      <inertial>
-      <origin rpy="0 0 0" xyz="0 0 0"/>
-      <mass value="0.05"/>
-      <inertia ixx="1" ixy="0.0" ixz="0.0" iyy="1" iyz="0.0" izz="1"/>
-    </inertial>
- </link>
-	<!-- GRIPPER LINKS -->
-  <link name="link_gripper_base">
-    <visual>
-      <origin rpy="0 0 0" xyz="0 0 -0.045"/>
-      <geometry>
-        <mesh filename="package://pa10_description/gripper_stl/pa10_gripper_base.stl"  scale="1 1 1"/>
-      </geometry>
-      <material name="">
-        <color rgba="0.2 0.2 0.2 1.0"/>
-      </material>
-    </visual>
-    <collision>
-      <origin rpy="0 0 0" xyz="0 0 -0.045"/>
-      <geometry>
-        <mesh filename="package://pa10_description/gripper_stl/pa10_gripper_base.stl"  scale="1 1 1"/>
-      </geometry>
-    </collision>
-    <inertial>
-      <origin rpy="0 0 0" xyz="0 0 -0.045"/>
-      <mass value="0.001"/>
-      <inertia ixx="1" ixy="0.0" ixz="0.0" iyy="1" iyz="0.0" izz="1"/>
-    </inertial>
-  </link>
-	<link name="link_finger_1">
-    <visual>
-      <origin rpy="-3.14159 -1.57079 0" xyz="-0.0225 0.075 -0.01"/>
-      <geometry>
-        <mesh filename="package://pa10_description/gripper_stl/finger.STL"  scale="0.001 0.001 0.001"/>
-      </geometry>
-      <material name="">
-        <color rgba="${255/255} ${108/255} ${10/255} 1.0"/>
-      </material>
-    </visual>
-    <collision>
-      <origin rpy="-3.14159 -1.57079 0" xyz="-0.0225 0.075 -0.01"/>
-      <geometry>
-        <mesh filename="package://pa10_description/gripper_stl/finger.STL"  scale="0.001 0.001 0.001"/>
-      </geometry>
-    </collision>
+      <xacro:inertia_cylinder height="0.05"  radius = "0.08" mass="0.5" axis="1"/>
+    </inertial>
+  </link>
+  <link name="link_wrist_3"/>
+  <link name="link_ee_tool">
     <inertial>
       <origin rpy="0 0 0" xyz="0 0 0"/>
       <mass value="0.1"/>
-      <inertia ixx="1" ixy="0.0" ixz="0.0" iyy="1" iyz="0.0" izz="1"/>
-    </inertial>
-  </link>
-	<link name="link_finger_2">
+      <inertia ixx="0.001" ixy="0.0" ixz="0.0" iyy="0.001" iyz="0.0" izz="0.001"/>
+    </inertial>
+  </link>
+  <!-- GRIPPER LINKS -->
+  <link name="link_gripper_base">
+    <visual>
+      <origin rpy="0 0 0" xyz="0 0 -0.045"/>
+      <geometry>
+        <mesh filename="package://pa10_description/gripper_stl/pa10_gripper_base.stl" scale="1 1 1"/>
+      </geometry>
+      <material name="">
+        <color rgba="0.2 0.2 0.2 1.0"/>
+      </material>
+    </visual>
+    <collision>
+      <origin rpy="0 0 0" xyz="0 0 -0.045"/>
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
File: pa10_description/urdf/pa10csl.gazebo.urdf.xacro (robot description, xacro)
@@ -15,4 +15,21 @@
     </plugin>
   </gazebo>
+  <!-- Inertial of Cylinder -->
+  <xacro:macro name="inertia_cylinder" params="mass height radius axis:=0">
+    <xacro:property name="Ir" value="${0.0833*mass*(3.0*radius*radius + height*height)}" />
+    <xacro:property name="Ih" value="${0.5*mass*(radius*radius)}" />
+    <!-- z Axis -->
+    <xacro:unless value="${axis}">
+      <inertia ixx="${Ir}" ixy="0" ixz="0" iyy="${Ir}" iyz="0" izz="${Ih}" />
+    </xacro:unless>
+    <!-- y Axis -->
+    <xacro:unless value="${axis-1}">
+      <inertia ixx="${Ir}" ixy="0" ixz="0" iyy="${Ih}" izz="${Ir}" iyz="0" />
+    </xacro:unless>
+    <!-- x Axis -->
+    <xacro:unless value="${axis-2}">
+      <inertia ixx="${Ih}" iyy="${Ir}" iyz="0" izz="${Ir}" ixy="0" ixz="0" />
+    </xacro:unless>
+  </xacro:macro>
   <!-- base_link -->
   <gazebo reference="base_link">
