Commit message: devel

File: pa10_description/urdf/materials.xacro (robot description, xacro)
@@ -1,4 +1,4 @@
 <?xml version="1.0"?>
-<robot>
+<robot xmlns:xacro="http://www.ros.org/wiki/xacro">
   <material name="black">
     <color rgba="0.0 0.0 0.0 1.0"/>

File: pa10_description/urdf/pa10_csl.urdf.xacro (robot description, xacro)
@@ -7,6 +7,8 @@
   <!-- namespace of the robot -->
   <xacro:arg name="interface" default="velocity"/>
-  <!-- namespace of the robot -->
+  <!-- camera -->
   <xacro:arg name="enable_camera" default="false"/>
+  <!-- color -->
+  <xacro:arg name="color" default="default"/>
   <xacro:property name="is_multiple" value="$(arg multiple)" />
   <xacro:property name="nsp" value="$(arg namespace)" />
@@ -17,11 +19,11 @@
   <!-- NOT THE ACTUAL VALUE -->
   <xacro:property name="arm_eps" value="0.02" />
-  <xacro:property name="joint_1_max_effort" value="150.0"/>
-  <xacro:property name="joint_2_max_effort" value="150.0"/>
-  <xacro:property name="joint_3_max_effort" value="150.0"/>
-  <xacro:property name="joint_4_max_effort" value="150.0"/>
-  <xacro:property name="joint_5_max_effort" value="150.0"/>
-  <xacro:property name="joint_6_max_effort" value="150.0"/>
-  <xacro:property name="joint_7_max_effort" value="150.0"/>
+  <xacro:property name="joint_1_max_effort" value="550.0"/>
+  <xacro:property name="joint_2_max_effort" value="550.0"/>
+  <xacro:property name="joint_3_max_effort" value="550.0"/>
+  <xacro:property name="joint_4_max_effort" value="550.0"/>
+  <xacro:property name="joint_5_max_effort" value="550.0"/>
+  <xacro:property name="joint_6_max_effort" value="550.0"/>
+  <xacro:property name="joint_7_max_effort" value="550.0"/>
   <!-- JOINTS POSITION LIMITS -->
   <!-- Real Values: [177, 94, 174, 137, 255, 165, 255] (deg)-->
@@ -35,6 +37,6 @@
   <!-- JOINTS VELOCITIE LIMITS-->
   <!-- Real Values: [1, 1, 2, 2, 2, 2*pi, 2*pi] (rad/sec)-->
-  <xacro:property name="joint_1_max_velocity" value="0.85"/>
-  <xacro:property name="joint_2_max_velocity" value="0.85"/>
+  <xacro:property name="joint_1_max_velocity" value="1.85"/>
+  <xacro:property name="joint_2_max_velocity" value="1.85"/>
   <xacro:property name="joint_3_max_velocity" value="1.85"/>
   <xacro:property name="joint_4_max_velocity" value="1.85"/>
@@ -455,3 +457,5 @@
   <xacro:arm_simple_transmission name="finger_joint_1" reduction="10" interface="velocity"/>
   <xacro:arm_simple_transmission name="finger_joint_2" reduction="10" interface="velocity"/>
+  <!-- COLORS GAZEBO -->
+  <xacro:gazebo_materials prefix="" color="$(arg color)" />
 </robot>

File: pa10_description/urdf/pa10_csl_ns.urdf.xacro (robot description, xacro)
@@ -1,219 +1,258 @@
 <?xml version="1.0" ?>
-<robot name="pa10"
+<root xmlns:xi="http://www.w3.org/2001/XInclude"
+  xmlns:gazebo="http://playerstage.sourceforge.net/gazebo/xmlschema/#gz"
+  xmlns:model="http://playerstage.sourceforge.net/gazebo/xmlschema/#model"
+  xmlns:sensor="http://playerstage.sourceforge.net/gazebo/xmlschema/#sensor"
+  xmlns:body="http://playerstage.sourceforge.net/gazebo/xmlschema/#body"
+  xmlns:geom="http://playerstage.sourceforge.net/gazebo/xmlschema/#geom"
+  xmlns:joint="http://playerstage.sourceforge.net/gazebo/xmlschema/#joint"
+  xmlns:controller="http://playerstage.sourceforge.net/gazebo/xmlschema/#controller"
+  xmlns:interface="http://playerstage.sourceforge.net/gazebo/xmlschema/#interface"
+  xmlns:rendering="http://playerstage.sourceforge.net/gazebo/xmlschema/#rendering"
+  xmlns:renderable="http://playerstage.sourceforge.net/gazebo/xmlschema/#renderable"
+  xmlns:physics="http://playerstage.sourceforge.net/gazebo/xmlschema/#physics"
   xmlns:xacro="http://www.ros.org/wiki/xacro">
-  <xacro:macro name="robotic_arm" params="name root_link tool_link interface:=velocity is_multiple:=false nsp:=''"/>
-      <xacro:property name="pi" value="3.1415926535897931" />
-      <!-- JOINTS EFFORT LIMITS -->
-      <!-- NOT THE ACTUAL VALUE -->
-      <xacro:property name="arm_eps" value="0.02" />
-      <xacro:property name="joint_1_max_effort" value="150.0"/>
-      <xacro:property name="joint_2_max_effort" value="150.0"/>
-      <xacro:property name="joint_3_max_effort" value="150.0"/>
-      <xacro:property name="joint_4_max_effort" value="150.0"/>
-      <xacro:property name="joint_5_max_effort" value="150.0"/>
-      <xacro:property name="joint_6_max_effort" value="150.0"/>
-      <xacro:property name="joint_7_max_effort" value="150.0"/>
-      <!-- JOINTS POSITION LIMITS -->
-      <!-- Real Values: [177, 94, 174, 137, 255, 165, 255] (deg)-->
-      <xacro:property name="joint_1_max_position" value="${170.0 *pi/180.0}"/>
-      <xacro:property name="joint_2_max_position" value="${90.0 *pi/180.0}"/>
-      <xacro:property name="joint_3_max_position" value="${170.0 *pi/180.0}"/>
-      <xacro:property name="joint_4_max_position" value="${130.0 *pi/180.0}"/>
-      <xacro:property name="joint_5_max_position" value="${250.0 *pi/180.0}"/>
-      <xacro:property name="joint_6_max_position" value="${160.0 *pi/180.0}"/>
-      <xacro:property name="joint_7_max_position" value="${250.0 *pi/180.0}"/>
-      <!-- JOINTS VELOCITIE LIMITS-->
-      <!-- Real Values: [1, 1, 2, 2, 2, 2*pi, 2*pi] (rad/sec)-->
-      <xacro:property name="joint_1_max_velocity" value="0.85"/>
-      <xacro:property name="joint_2_max_velocity" value="0.85"/>
-      <xacro:property name="joint_3_max_velocity" value="1.85"/>
-      <xacro:property name="joint_4_max_velocity" value="1.85"/>
-      <xacro:property name="joint_5_max_velocity" value="1.85"/>
-      <xacro:property name="joint_6_max_velocity" value="${1.8*pi}"/>
-      <xacro:property name="joint_7_max_velocity" value="${1.8*pi}"/>
-      <!-- JOINT DYNAMICS DAMPING + FRICTION-->
-      <!-- >> !! Not Real Values !! << -->
-      <!-- DAMPING -->
-      <xacro:property name="joint_1_damping" value="0.8"/>
-      <xacro:property name="joint_2_damping" value="0.8"/>
-      <xacro:property name="joint_3_damping" value="0.8"/>
-      <xacro:property name="joint_4_damping" value="0.8"/>
-      <xacro:property name="joint_5_damping" value="0.8"/>
-      <xacro:property name="joint_6_damping" value="0.8"/>
-      <xacro:property name="joint_7_damping" value="0.8"/>
-      <!-- FRICTION -->
-      <xacro:property name="joint_1_friction" value="0.1"/>
-      <xacro:property name="joint_2_friction" value="0.1"/>
-      <xacro:property name="joint_3_friction" value="0.1"/>
-      <xacro:property name="joint_4_friction" value="0.1"/>
-      <xacro:property name="joint_5_friction" value="0.1"/>
-      <xacro:property name="joint_6_friction" value="0.1"/>
-      <xacro:property name="joint_7_friction" value="0.1"/>
-      <!-- Import all Gazebo-customization elements, including Gazebo colors -->
-      <xacro:include filename="$(find pa10_description)/urdf/pa10csl.gazebo.urdf.xacro" />
-      <!-- Import Rviz colors -->
-      <xacro:include filename="$(find pa10_description)/urdf/materials.xacro" />
-      <!-- Import Transmitions -->
-      <xacro:include filename="$(find pa10_description)/urdf/arm.transmission.xacro"/>
-      <link name="${name}base_link">
+  <xacro:property name="is_multiple" value="false" />
+  <xacro:property name="nsp" value="" />
+  <xacro:property name="pi" value="3.1415926535897931" />
+  <!-- Import all Gazebo-customization elements, including Gazebo colors -->
+  <xacro:include filename="$(find pa10_description)/urdf/pa10csl.gazebo.urdf.xacro" />
+  <!-- Import Transmitions -->
+  <xacro:include filename="$(find pa10_description)/urdf/arm.transmission.xacro"/>
+  <xacro:macro name="pa10_arm" params="prefix root_link:=None tool_link:='link_ee_tool' interface:=velocity enable_camera:=false color:='default'">
+    <xacro:property name="HWInterface" value="${interface}" />
+    <xacro:property name="enable_camera_" value="${enable_camera}" />
+    <!-- JOINTS EFFORT LIMITS -->
+    <!-- NOT THE ACTUAL VALUE -->
+    <xacro:property name="arm_eps" value="0.02" />
+    <xacro:property name="joint_1_max_effort" value="550.0"/>
+    <xacro:property name="joint_2_max_effort" value="550.0"/>
+    <xacro:property name="joint_3_max_effort" value="550.0"/>
+    <xacro:property name="joint_4_max_effort" value="550.0"/>
+    <xacro:property name="joint_5_max_effort" value="550.0"/>
+    <xacro:property name="joint_6_max_effort" value="550.0"/>
+    <xacro:property name="joint_7_max_effort" value="550.0"/>
+    <!-- JOINTS POSITION LIMITS -->
+    <!-- Real Values: [177, 94, 174, 137, 255, 165, 255] (deg)-->
+    <xacro:property name="joint_1_max_position" value="${170.0 *pi/180.0}"/>
+    <xacro:property name="joint_2_max_position" value="${90.0 *pi/180.0}"/>
+    <xacro:property name="joint_3_max_position" value="${170.0 *pi/180.0}"/>
+    <xacro:property name="joint_4_max_position" value="${130.0 *pi/180.0}"/>
+    <xacro:property name="joint_5_max_position" value="${250.0 *pi/180.0}"/>
+    <xacro:property name="joint_6_max_position" value="${160.0 *pi/180.0}"/>
+    <xacro:property name="joint_7_max_position" value="${250.0 *pi/180.0}"/>
+    <!-- JOINTS VELOCITIE LIMITS-->
+    <!-- Real Values: [1, 1, 2, 2, 2, 2*pi, 2*pi] (rad/sec)-->
+    <xacro:property name="joint_1_max_velocity" value="1.85"/>
+    <xacro:property name="joint_2_max_velocity" value="1.85"/>
+    <xacro:property name="joint_3_max_velocity" value="2.85"/>
+    <xacro:property name="joint_4_max_velocity" value="2.85"/>
+    <xacro:property name="joint_5_max_velocity" value="2.85"/>
+    <xacro:property name="joint_6_max_velocity" value="${2.8*pi}"/>
+    <xacro:property name="joint_7_max_velocity" value="${2.8*pi}"/>
+    <!-- JOINT DYNAMICS DAMPING + FRICTION-->
+    <!-- >> !! Not Real Values !! << -->
+    <!-- DAMPING -->
+    <xacro:property name="joint_1_damping" value="0.8"/>
+    <xacro:property name="joint_2_damping" value="0.8"/>
+    <xacro:property name="joint_3_damping" value="0.8"/>
+    <xacro:property name="joint_4_damping" value="0.8"/>
+    <xacro:property name="joint_5_damping" value="0.8"/>
+    <xacro:property name="joint_6_damping" value="0.8"/>
+    <xacro:property name="joint_7_damping" value="0.8"/>
+    <xacro:property name="joint_finger_damping" value="0.8"/>
+    <!-- FRICTION -->
+    <xacro:property name="joint_1_friction" value="0.1"/>
+    <xacro:property name="joint_2_friction" value="0.1"/>
+    <xacro:property name="joint_3_friction" value="0.1"/>
+    <xacro:property name="joint_4_friction" value="0.1"/>
+    <xacro:property name="joint_5_friction" value="0.1"/>
+    <xacro:property name="joint_6_friction" value="0.1"/>
+    <xacro:property name="joint_7_friction" value="0.1"/>
+    <xacro:property name="joint_finger_friction" value="0.1"/>
+    <xacro:if value="${enable_camera_}">
+      <link name="${prefix}kinect2_rgb_optical_frame">
         <visual>
-          <origin rpy="0 0 3.14" xyz="0 0 0"/>
+          <origin rpy="${pi} ${-pi/2.0} ${-pi/2.0}" xyz="0 0 0"/>
           <geometry>
-            <mesh filename="package://pa10_description/pa10_stl/S1.stl" scale="1 1 1"/>
+            <mesh filename="package://pa10_description/sensors_3D_models/kinect.dae" scale="1 1 1"/>
           </geometry>
-          <material name="pa10_blue">
+          <material name="">
+            <color rgba="0.0 0.0 0.0 1.0"/>
           </material>
         </visual>
         <collision>
-          <origin rpy="0 0 3.14" xyz="0 0 0"/>
+          <origin rpy="${pi} ${-pi/2.0} ${-pi/2.0}" xyz="0 0 0"/>
           <geometry>
-            <mesh filename="package://pa10_description/pa10_stl_collision/S1_collision.stl" scale="1 1 1"/>
+            <mesh filename="package://pa10_description/sensors_3D_models/kinect.dae" scale="1 1 1"/>
           </geometry>
         </collision>
         <inertial>
-          <origin rpy="0 0 3.14" xyz="0 0 0"/>
+          <origin rpy="0 0 0" xyz="0 0 1"/>
           <mass value="0.5"/>
-          <inertia ixx="1" ixy="0.0" ixz="0.0" iyy="1" iyz="0.0" izz="1"/>
+          <inertia ixx="0.001" ixy="0.0" ixz="0.0" iyy="0.001" iyz="0.0" izz="0.001"/>
         </inertial>
       </link>
-      <link name="${name}link_shoulder_1">
-        <visual>
-          <origin rpy="0 0 0" xyz="0 0 0.117"/>
-          <geometry>
-            <mesh filename="package://pa10_description/pa10_stl/S2.stl" scale="1 1 1"/>
-          </geometry>
-          <material name="">
-            <color rgba="0.13 0.13 0.13 1.0"/>
-          </material>
-        </visual>
-        <collision>
-          <origin rpy="0 0 0" xyz="0 0 0.117"/>
-          <geometry>
-            <mesh filename="package://pa10_description/pa10_stl_collision/S2_collision.stl" scale="1 1 1"/>
-          </geometry>
-        </collision>
-        <inertial>
-          <origin rpy="0 0 0" xyz="0 0 0.117"/>
-          <mass value="0.5"/>
-          <inertia ixx="1" ixy="0.0" ixz="0.0" iyy="1" iyz="0.0" izz="1"/>
-        </inertial>
-      </link>
-      <link name="${name}link_shoulder_2">
-        <visual>
-          <origin rpy="-1.57079 0 3.14159" xyz="0 0 0"/>
-          <geometry>
-            <mesh filename="package://pa10_description/pa10_stl/S3.stl" scale="1 1 1"/>
-          </geometry>
-          <material name="pa10_blue">
-          </material>
-        </visual>
-        <collision>
-          <origin rpy="-1.57079 0 3.14159" xyz="0 0 0"/>
-          <geometry>
-            <mesh filename="package://pa10_description/pa10_stl_collision/S3_collision.stl" scale="1 1 1"/>
-          </geometry>
-        </collision>
-        <inertial>
-          <origin rpy="-1.57079 0 3.14159" xyz="0 0 0"/>
-          <mass value="0.5"/>
-          <inertia ixx="1" ixy="0.0" ixz="0.0" iyy="1" iyz="0.0" izz="1"/>
-        </inertial>
-      </link>
-      <link name="${name}link_shoulder_to_elbow">
-        <inertial>
-          <origin rpy="0 0 0" xyz="0 0 1"/>
-          <mass value="0.5"/>
-          <inertia ixx="1" ixy="0.0" ixz="0.0" iyy="1" iyz="0.0" izz="1"/>
-        </inertial>
-      </link>
-      <link name="${name}link_elbow_1">
-        <visual>
-          <origin rpy="0 0 0" xyz="0 0.0 0.133"/>
-          <geometry>
-            <mesh filename="package://pa10_description/pa10_stl/E1.stl" scale="1 1 1"/>
-          </geometry>
-          <material name="">
-            <color rgba="0.13 0.13 0.13 1.5"/>
-          </material>
-        </visual>
-        <collision>
-          <origin rpy="0 0 0" xyz="0 0.0 0.133"/>
-          <geometry>
-            <mesh filename="package://pa10_description/pa10_stl_collision/E1_collision.stl" scale="1 1 1"/>
-          </geometry>
-        </collision>
-        <inertial>
-          <origin rpy="0 0 0" xyz="0 0.0 0.133"/>
-          <mass value="0.5"/>
-          <inertia ixx="1" ixy="0.0" ixz="0.0" iyy="1" iyz="0.0" izz="1"/>
-        </inertial>
-      </link>
-      <link name="${name}link_elbow_2">
-        <visual>
-          <origin rpy="1.57079 0 0" xyz="0 0.003 0"/>
-          <geometry>
-            <mesh filename="package://pa10_description/pa10_stl/E2.stl" scale="1 1 1"/>
-          </geometry>
-          <material name="">
-            <color rgba="0.34 0.35 0.36 1.0"/>
-          </material>
-        </visual>
-        <collision>
-          <origin rpy="-1.57079 0 0" xyz="0 0.003 0"/>
-          <geometry>
-            <mesh filename="package://pa10_description/pa10_stl_collision/E2_collision.stl" scale="1 1 1"/>
-          </geometry>
-        </collision>
-        <inertial>
-          <origin rpy="1.57079 0 0" xyz="0 0.003 0"/>
-          <mass value="0.5"/>
-          <inertia ixx="1" ixy="0.0" ixz="0.0" iyy="1" iyz="0.0" izz="1"/>
-        </inertial>
-      </link>
-      <link name="${name}link_wrist_1">
-        <visual>
-          <origin rpy="0 0 0" xyz="0 0 0.195"/>
-          <geometry>
-            <mesh filename="package://pa10_description/pa10_stl/W1.stl" scale="1 1 1"/>
-          </geometry>
-          <material name="">
-            <color rgba="0.13 0.13 0.13 1.5"/>
-          </material>
-        </visual>
-        <collision>
-          <origin rpy="0 0 0" xyz="0 0 0.195"/>
-          <geometry>
-            <mesh filename="package://pa10_description/pa10_stl_collision/W1_collision.stl" scale="1 1 1"/>
-          </geometry>
-        </collision>
-        <inertial>
-          <origin rpy="0 0 0" xyz="0 0 0.195"/>
-          <mass value="0.5"/>
-          <inertia ixx="1" ixy="0.0" ixz="0.0" iyy="1" iyz="0.0" izz="1"/>
-        </inertial>
-      </link>
-      <link name="${name}link_wrist_2">
-        <visual>
-          <origin rpy="1.57079 0 0" xyz="0 0 0"/>
-          <geometry>
-            <mesh filename="package://pa10_description/pa10_stl/W2.stl" scale="1 1 1"/>
-          </geometry>
-          <material name="pa10_blue">
-          </material>
-        </visual>
-        <collision>
-          <origin rpy="1.57079 0 0" xyz="0 0 0"/>
-          <geometry>
-            <mesh filename="package://pa10_description/pa10_stl_collision/W2_collision.stl" scale="1 1 1"/>
-          </geometry>
-        </collision>
-        <inertial>
-          <origin rpy="1.57079 0 0" xyz="0 0 0"/>
-          <mass value="0.5"/>
-          <inertia ixx="1" ixy="0.0" ixz="0.0" iyy="1" iyz="0.0" izz="1"/>
-        </inertial>
-      </link>
-      <link name="${name}link_wrist_3"/>
-      <!-- <link name="link_ee_tool">
+      <link name="${prefix}kinect2_ir_optical_frame"/>
+    </xacro:if>
+    <link name="${prefix}base_link">
+      <visual>
+        <origin rpy="0 0 3.14" xyz="0 0 0"/>
+        <geometry>
+          <mesh filename="package://pa10_description/pa10_stl/S1.stl" scale="1 1 1"/>
+        </geometry>
+        <material name="pa10_blue">
+        </material>
+      </visual>
+      <collision>
+        <origin rpy="0 0 3.14" xyz="0 0 0"/>
+        <geometry>
+          <mesh filename="package://pa10_description/pa10_stl_collision/S1_collision.stl" scale="1 1 1"/>
+        </geometry>
+      </collision>
+      <inertial>
+        <origin rpy="0 0 3.14" xyz="0 0 0.1"/>
+        <mass value="0.5"/>
+        <xacro:inertia_cylinder height="0.2"  radius = "0.1" mass="0.5"/>
+      </inertial>
+    </link>
+    <link name="${prefix}link_shoulder_1">
+      <visual>
+        <origin rpy="0 0 0" xyz="0 0 0.117"/>
+        <geometry>
+          <mesh filename="package://pa10_description/pa10_stl/S2.stl" scale="1 1 1"/>
+        </geometry>
+        <material name="">
+          <color rgba="0.88 0.88 0.88 1.0"/>
+        </material>
+      </visual>
+      <collision>
+        <origin rpy="0 0 0" xyz="0 0 0.117"/>
+        <geometry>
+          <mesh filename="package://pa10_description/pa10_stl_collision/S2_collision.stl" scale="1 1 1"/>
+        </geometry>
+      </collision>
+      <inertial>
+        <origin rpy="0 0 0" xyz="0 0 0.117"/>
+        <mass value="0.5"/>
+        <xacro:inertia_cylinder height="0.12"  radius = "0.08" mass="0.5"/>
+      </inertial>
+    </link>
+    <link name="${prefix}link_shoulder_2">
+      <visual>
+        <origin rpy="-1.57079 0 3.14159" xyz="0 0 0"/>
+        <geometry>
+          <mesh filename="package://pa10_description/pa10_stl/S3.stl" scale="1 1 1"/>
+        </geometry>
+        <material name="pa10_blue">
+        </material>
+      </visual>
+      <collision>
+        <origin rpy="-1.57079 0 3.14159" xyz="0 0 0"/>
+        <geometry>
+          <mesh filename="package://pa10_description/pa10_stl_collision/S3_collision.stl" scale="1 1 1"/>
+        </geometry>
+      </collision>
+      <inertial>
+        <origin rpy="-1.57079 0 3.14159" xyz="0 -0.22 0.0"/>
+        <mass value="0.5"/>
+        <xacro:inertia_cylinder height="0.18"  radius = "0.05" mass="0.5" axis="0"/>
+      </inertial>
+    </link>
+    <link name="${prefix}link_shoulder_to_elbow">
+      <inertial>
+        <origin rpy="0 0 0" xyz="0 0 0.22"/>
+        <mass value="0.5"/>
+        <inertia ixx="0.001" ixy="0.0" ixz="0.0" iyy="0.001" iyz="0.0" izz="0.001"/>
+      </inertial>
+    </link>
+    <link name="${prefix}link_elbow_1">
+      <visual>
+        <origin rpy="0 0 0" xyz="0 0.0 0.133"/>
+        <geometry>
+          <mesh filename="package://pa10_description/pa10_stl/E1.stl" scale="1 1 1"/>
+        </geometry>
+        <material name="">
+          <color rgba="0.88 0.88 0.88 1.5"/>
+        </material>
+      </visual>
+      <collision>
+        <origin rpy="0 0 0" xyz="0 0.0 0.133"/>
+        <geometry>
+          <mesh filename="package://pa10_description/pa10_stl_collision/E1_collision.stl" scale="1 1 1"/>
+        </geometry>
+      </collision>
+      <inertial>
+        <origin rpy="0 0 0" xyz="0 0.0 0.133"/>
+        <mass value="0.5"/>
+        <xacro:inertia_cylinder height="0.12"  radius = "0.08" mass="0.5"/>
+      </inertial>
+    </link>
+    <link name="${prefix}link_elbow_2">
+      <visual>
+        <origin rpy="1.57079 0 0" xyz="0 0.003 0"/>
+        <geometry>
+          <mesh filename="package://pa10_description/pa10_stl/E2.stl" scale="1 1 1"/>
+        </geometry>
+        <material name="pa10_blue">
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