Commit message: cooperative multi robot simulation

File: pa10_description/urdf/cooperative_pa10.urdf.xacro (robot description, xacro)
@@ -1,129 +1,192 @@
 <?xml version="1.0" ?>
 <robot name="pa10"
-    xmlns:xacro="http://www.ros.org/wiki/xacro">
-    <xacro:arg name="interface" default="velocity"/>
-    <xacro:property name="HWInterface" value="$(arg interface)" />
-    <!-- Include PA10 CSL Namespace  -->
-    <xacro:include filename="$(find pa10_description)/urdf/pa10_csl_ns.urdf.xacro"/>
-    <link name="world"/>
-    <!-- PA10 1 Links - Joints -->
-    <link name="pa10_1_root_link">
-        <inertial>
-            <origin rpy="0 0 0" xyz="0 0 0"/>
-            <mass value="1.5"/>
-            <inertia ixx="1" ixy="0.0" ixz="0.0" iyy="1" iyz="0.0" izz="1"/>
-        </inertial>
+  xmlns:xacro="http://www.ros.org/wiki/xacro">
+  <xacro:arg name="multiple" default="false"/>
+  <!-- If multiple robots will be used -->
+  <xacro:arg name="namespace" default=""/>
+  <!-- namespace of the robot -->
+  <!-- camera -->
+  <xacro:arg name="enable_camera" default="false"/>
+  <xacro:arg name="num_of_agents" default="3"/>
+  <!-- robot arguements -->
+  <xacro:arg name="pa10_1_color" default="default"/>
+  <xacro:arg name="robot_1_interface" default="velocity"/>
+  <xacro:arg name="pa10_2_color" default="red"/>
+  <xacro:arg name="robot_2_interface" default="velocity"/>
+  <xacro:arg name="pa10_3_color" default="green"/>
+  <xacro:arg name="robot_3_interface" default="velocity"/>
+  <xacro:arg name="use_object" default="true"/>
+  <xacro:arg name="type_of_object" default="box"/>
+  <!-- Number of Agents -->
+  <xacro:property name="agents" value="$(arg num_of_agents)"/>
+  <!-- general properties -->
+  <xacro:property name="robot_radius" value="0.938"/>
+  <xacro:property name="cos30" value="0.866"/>
+  <xacro:property name="sin30" value="0.5"/>
+  <!-- ROBOT 1 Properties -->
+  <xacro:property name="robot_1_x" value="0.0"/>
+  <xacro:property name="robot_1_y" value="-1.1"/>
+  <xacro:property name="robot_1_yaw" value= "1.57079"/>
+  <xacro:property name="HWInterface" value="$(arg robot_1_interface)" />
+  <!-- ROBOT 2 Properties -->
+  <xacro:property name="robot_2_enable" value="false"/>
+  <xacro:property name="robot_2_x" value="0.5"/>
+  <xacro:property name="robot_2_y" value="1.1"/>
+  <xacro:property name="robot_2_yaw" value="1.57079"/>
+  <xacro:property name="HWInterface2" value="$(arg robot_2_interface)" />
+  <!-- ROBOT 3 Properties -->
+  <xacro:property name="robot_3_enable" value="false"/>
+  <xacro:property name="robot_3_x" value="-0.5"/>
+  <xacro:property name="robot_3_y" value="1.1"/>
+  <xacro:property name="robot_3_yaw" value="1.57079"/>
+  <xacro:property name="HWInterface3" value="$(arg robot_3_interface)" />
+  <xacro:property name="is_multiple" value="$(arg multiple)" />
+  <xacro:property name="nsp" value="$(arg namespace)" />
+  <xacro:property name="enable_camera_" value="$(arg enable_camera)" />
+  <!-- OBJECT PARAMETERS -->
+  <xacro:property name="use_object_" value="$(arg use_object)"/>
+  <xacro:property name="object_length" value="0.545"/>
+  <xacro:property name="object_height" value="0.545"/>
+  <xacro:property name="object_color" value="white"/>
+  <xacro:property name="object_mass" value="1.0"/>
+  <xacro:property name="object_type" value="$(arg type_of_object)"/>
+  <!-- Import all Gazebo-customization elements, including Gazebo colors -->
+  <xacro:include filename="$(find pa10_description)/urdf/pa10csl.gazebo.urdf.xacro" />
+  <!-- Import Rviz colors -->
+  <xacro:include filename="$(find pa10_description)/urdf/materials.xacro" />
+  <!-- Import Transmitions -->
+  <xacro:include filename="$(find pa10_description)/urdf/arm.transmission.xacro"/>
+  <!-- Import pa10 properties -->
+  <xacro:include filename="$(find pa10_description)/urdf/pa10properties.xacro"/>
+  <!-- Import sensors -->
+  <xacro:include filename="$(find pa10_description)/urdf/sensors.urdf.xacro"/>
+  <!-- Import PA10 Arm -->
+  <xacro:include filename="$(find pa10_description)/urdf/pa10root.urdf.xacro"/>
+  <xacro:if value="${agents == 2}">
+    <xacro:if value="${object_type == 'box'}">
+      <xacro:property name="robot_2_x" value="0.0"/>
+      <xacro:property name="robot_2_enable" value="true"/>
+      <xacro:property name="robot_3_enable" value="false"/>
+      <xacro:property name="object_length" value="0.545"/>
+      <xacro:property name="use_object_" value="true"/>
+    </xacro:if>
+    <xacro:if value="${object_type == 'cylinder'}">
+      <xacro:property name="robot_2_x" value="0.0"/>
+      <xacro:property name="robot_2_enable" value="true"/>
+      <xacro:property name="robot_3_enable" value="false"/>
+      <xacro:property name="object_length" value="${0.545/2}"/>
+      <xacro:property name="use_object_" value="true"/>
+    </xacro:if>
+  </xacro:if>
+  <xacro:if value="${agents == 3}">
+    <xacro:if value="${object_type == 'cylinder'}">
+      <xacro:property name="object_length" value="${0.545/2}"/>
+      <xacro:property name="use_object_" value="true"/>
+      <xacro:property name="robot_2_x" value="${cos30*(object_length + robot_radius-0.1)}"/>
+      <xacro:property name="robot_2_y" value="${sin30*(object_length + robot_radius-0.1)}"/>
+      <xacro:property name="robot_2_yaw" value="${pi/6}"/>
+      <xacro:property name="robot_2_enable" value="true"/>
+      <xacro:property name="robot_3_x" value="${-cos30*(object_length + robot_radius-0.1)}"/>
+      <xacro:property name="robot_3_y" value="${sin30*(object_length + robot_radius-0.1)}"/>
+      <xacro:property name="robot_3_yaw" value="${pi/3+pi/2}"/>
+      <xacro:property name="robot_3_enable" value="true"/>
+    </xacro:if>
+    <xacro:if value="${object_type == 'box'}">
+      <xacro:property name="use_object_" value="true"/>
+      <xacro:property name="object_length" value="1.345"/>
+      <xacro:property name="robot_2_x" value="0.5"/>
+      <xacro:property name="robot_2_enable" value="true"/>
+      <xacro:property name="robot_3_x" value="-0.5"/>
+      <xacro:property name="robot_3_enable" value="true"/>
+    </xacro:if>
+  </xacro:if>
+  <!-- LINKS -->
+  <link name="world"/>
+  <xacro:pa10_arm prefix="pa10_1_" xyz="${robot_1_x} ${robot_1_y} 0.0" rpy="0 0 ${robot_1_yaw}" S2_offset="0.5" E2_offset="0.53" W2_offset="0.54" W3_offset="-1.57" interface="${HWInterface}" enable_camera="false" color="$(arg pa10_1_color)"/>
+  <xacro:if value="${use_object_}">
+    <!--- Object -->
+    <link name="object">
+      <visual>
+        <origin xyz="0 0 -0.0" rpy="0 0 0"/>
+        <geometry>
+          <xacro:if value="${object_type == 'cylinder'}">
+            <cylinder length="0.06" radius="${object_length}"/>
+          </xacro:if>
+          <xacro:if value="${object_type == 'box'}">
+            <box size="${object_length} ${object_height} 0.06"/>
+          </xacro:if>
+        </geometry>
+        <material name="orange"/>
+      </visual>
+      <collision>
+        <origin xyz="0 0 0.0" rpy="0 0 0"/>
+        <geometry>
+          <xacro:if value="${object_type == 'cylinder'}">
+            <cylinder length="0.06" radius="${object_length/1.2}"/>
+          </xacro:if>
+          <xacro:if value="${object_type == 'box'}">
+            <box size="${object_length/2} ${object_height/2} 0.06"/>
+          </xacro:if>
+        </geometry>
+      </collision>
+      <inertial>
+        <mass value="${object_mass}"/>
+        <xacro:if value="${object_type == 'cylinder'}">
+          <xacro:inertia_cylinder radius="${object_length}" height="0.06" mass="${object_mass}"/>
+        </xacro:if>
+        <xacro:if value="${object_type == 'box'}">
+          <xacro:inertia_box height="${object_length}" mass="${object_mass}"/>
+        </xacro:if>
+      </inertial>
     </link>
-    <link name="pa10_1_link_ee_tool">
-        <inertial>
-            <origin rpy="0 0 0" xyz="0 0 0"/>
-            <mass value="0.1"/>
-            <inertia ixx="0.001" ixy="0.0" ixz="0.0" iyy="0.001" iyz="0.0" izz="0.001"/>
-        </inertial>
-    </link>
-    <joint name="pa10_1_base_to_root" type="fixed">
-        <origin rpy="0 0 0" xyz="0 -1 0"/>
-        <parent link="world"/>
-        <child link="pa10_1_root_link"/>
+    <!-- Attach object to pa10_1 -->
+    <joint name="$pa10_1_ee_tool_to_object" type="fixed">
+      <origin rpy="1.576 0 -3.141" xyz="0 0 0.162"/>
+      <parent link="pa10_1_link_ee_tool"/>
+      <child link="object"/>
     </joint>
-    <xacro:pa10_arm prefix="pa10_1_" root_link="pa10_1_root_link" tool_link="pa10_1_link_ee_tool" interface="${HWInterface}" color="default"/>
-    <!-- PA10 2 Links - Joints -->
-    <link name="pa10_2_root_link">
-        <inertial>
-            <origin rpy="0 0 0" xyz="0 0 0"/>
-            <mass value="1.5"/>
-            <inertia ixx="1" ixy="0.0" ixz="0.0" iyy="1" iyz="0.0" izz="1"/>
-        </inertial>
-    </link>
-    <link name="pa10_2_link_ee_tool">
-        <inertial>
-            <origin rpy="0 0 0" xyz="0 0 0"/>
-            <mass value="0.1"/>
-            <inertia ixx="0.001" ixy="0.0" ixz="0.0" iyy="0.001" iyz="0.0" izz="0.001"/>
-        </inertial>
-    </link>
-    <joint name="pa10_2_base_to_root" type="fixed">
-        <origin rpy="0 0 0" xyz="0 1 0"/>
-        <parent link="world"/>
-        <child link="pa10_2_root_link"/>
-    </joint>
-    <xacro:pa10_arm prefix="pa10_2_" root_link="pa10_2_root_link" tool_link="pa10_2_link_ee_tool" interface="effort" color="red"/>
-    <link name="object_handle_2">
-        <inertial>
-            <origin rpy="0 0 0" xyz="0 0 0"/>
-            <mass value="0.1"/>
-            <inertia ixx="0.001" ixy="0.0" ixz="0.0" iyy="0.001" iyz="0.0" izz="0.001"/>
-        </inertial>
-    </link>
-    <!-- Object -->
-    <link name="common_object">
-        <visual>
-            <origin xyz="0 0 0" rpy="0 0 0" />
-            <geometry>
-                <box size="0.06 0.35 0.3" />
-            </geometry>
-            <material name="Cyan">
-                <color rgba="0 1.0 1.0 1.0"/>
-            </material>
-        </visual>
-        <collision>
-            <origin xyz="0 0 0" rpy="0 0 0"/>
-            <geometry>
-                <box size="0.06 0.24 0.25" />
-            </geometry>
-        </collision>
-        <inertial>
-            <origin rpy="0 0 0" xyz="0 0 0"/>
-            <mass value="0.5"/>
-            <inertia ixx="0.1" ixy="0.0" ixz="0.0" iyy="0.1" iyz="0.0" izz="0.1"/>
-        </inertial>
-    </link>
-    <!-- <gazebo>
-        <joint name="constrainted_multi_robot_joint" type="fixed">
-            <parent>pa10_1_link_ee_tool</parent>
-            <child>pa10_2_link_ee_tool</child>
-            <pose>0.00 0.5 0 0 0 0</pose>
-        </joint>
-    </gazebo>  -->
-    <joint name="pa10_1_to_object" type="fixed">
-        <!-- <parent>pa10_1_link_ee_tool</parent>
-            <child>common_object</child> -->
-        <!-- <origin>0.00 0.0 0.151 1.579 0 -1.543</origin> -->
-        <origin rpy="1.579 0 -1.543" xyz=" 0.00 0.0 0.151"/>
-        <parent link="pa10_1_link_ee_tool"/>
-        <child link="common_object"/>
-    </joint>
-    <joint name="object_to_pa10_2" type="fixed">
-        <origin rpy="-1.868 -1.505 -2.812" xyz=" 0.00 0.12 0.0"/>
-        <parent link="common_object"/>
-        <child link="object_handle_2"/>
-    </joint>
-    <!-- <gazebo>
-        <joint name="pa10_2_to_object" type="fixed">
-            <origin>0.00 0.0 0.121 -1.579 0.0 -1.633</origin>
-            <parent>pa10_2_link_ee_tool</parent>
-            <child>common_object</child>
-        </joint>
-    </gazebo> -->
-    <!-- <gazebo>
-        <joint name="pa10_2_to_object" type="fixed">
-            <parent>object_handle_2</parent>
-            <child>pa10_2_link_ee_tool</child>
-            <pose>0 0 0 0 0 0</pose>
-        </joint>
-    </gazebo>  -->
-    <!-- <gazebo>
-        <plugin name="Myrobot_ClosedLoopPlugin" filename="libpegasus_gazebo_closed_loop_plugin.so">
-            <joint>add_joint</joint>
-            <child>pa10_1_link_wrist_3</child>
-            <parent>pa10_2_link_wrist_3</parent>
-            <position>-0.024, -0.003, 0.729</position>
-            <rotation>-3.114, 0.032, 3.109</rotation>
-        </plugin>
-    </gazebo> -->
-    <!-- <joint name="pa10_2_to_object" type="fixed">
-        <parent link="object_handle_2"/>
-        <child link="pa10_2_link_ee_tool"/>
-        <origin rpy="0.0 0.0 0.0" xyz=" 0.00 0.0 0.0"/>
-    </joint> -->
+  </xacro:if>
+  <!-- ROBOT 2 -->
+  <xacro:if value="${robot_2_enable}">
+    <xacro:pa10_arm prefix="pa10_2_" xyz="${robot_2_x} ${robot_2_y} 0.0" rpy="0 0 ${robot_2_yaw}" S2_offset="-0.5" E2_offset="-0.53" W2_offset="-0.54" W3_offset="-1.57" interface="${HWInterface2}" enable_camera="false" color="$(arg pa10_2_color)"/>
+    <gazebo>
+      <joint name="object_to_pa10_2" type="fixed">
+        <parent>object</parent>
+        <child>pa10_2_link_ee_tool</child>
+        <xacro:if value="${object_type == 'cylinder'}">
+          <xacro:if value="${agents == 3}">
+            <!-- <pose>${robot_2_x-(cos30*robot_radius)} ${robot_2_y-(sin30*robot_radius)} 0.0 -1.576 0 2.094</pose> -->
+            <pose>0.157 0.102 -0.003 -1.571 0 2.094</pose>
+          </xacro:if>
+          <xacro:if value="${agents == 2}">
+            <pose>${robot_2_x} 0.162 0.0 -1.576 0 -3.142</pose>
+          </xacro:if>
+        </xacro:if>
+        <xacro:if value="${object_type == 'box'}">
+          <pose>${robot_2_x} 0.162 0.0 -1.576 0 -3.142</pose>
+        </xacro:if>
+      </joint>
+    </gazebo>
+  </xacro:if>
+  <!-- ROBOT 3 -->
+  <xacro:if value="${robot_3_enable}">
+    <xacro:pa10_arm prefix="pa10_3_" xyz="${robot_3_x} ${robot_3_y} 0.0" rpy="0 0 ${robot_3_yaw}" S2_offset="-0.5" E2_offset="-0.53" W2_offset="-0.54" W3_offset="-1.57" interface="${HWInterface3}" enable_camera="${enable_camera_}" color="$(arg pa10_3_color)"/>
+    <gazebo>
+      <joint name="object_to_pa10_3" type="fixed">
+        <parent>object</parent>
+        <child>pa10_3_link_ee_tool</child>
+        <xacro:if value="${object_type == 'cylinder'}">
+          <xacro:if value="${agents == 3}">
+            <pose>-0.157 0.102 -0.003 -1.571 0 -2.094</pose>
+          </xacro:if>
+          <xacro:if value="${agents == 2}">
+            <pose>${robot_3_x} 0.162 0.0 -1.576 0 -3.142</pose>
+          </xacro:if>
+        </xacro:if>
+        <xacro:if value="${object_type == 'box'}">
+          <pose>${robot_3_x} 0.162 0.0 -1.576 0 -3.142</pose>
+        </xacro:if>
+      </joint>
+    </gazebo>
+  </xacro:if>
 </robot>
