Commit message: cooperative multi robot simulation

File: pa10_description/urdf/pa10_csl.urdf.xacro (robot description, xacro)
@@ -15,53 +15,6 @@
   <xacro:property name="HWInterface" value="$(arg interface)" />
   <xacro:property name="enable_camera_" value="$(arg enable_camera)" />
-  <xacro:property name="pi" value="3.1415926535897931" />
-  <!-- JOINTS EFFORT LIMITS -->
-  <!-- NOT THE ACTUAL VALUE -->
-  <xacro:property name="arm_eps" value="0.02" />
-  <xacro:property name="joint_1_max_effort" value="550.0"/>
-  <xacro:property name="joint_2_max_effort" value="550.0"/>
-  <xacro:property name="joint_3_max_effort" value="550.0"/>
-  <xacro:property name="joint_4_max_effort" value="550.0"/>
-  <xacro:property name="joint_5_max_effort" value="550.0"/>
-  <xacro:property name="joint_6_max_effort" value="550.0"/>
-  <xacro:property name="joint_7_max_effort" value="550.0"/>
-  <!-- JOINTS POSITION LIMITS -->
-  <!-- Real Values: [177, 94, 174, 137, 255, 165, 255] (deg)-->
-  <xacro:property name="joint_1_max_position" value="${170.0 *pi/180.0}"/>
-  <xacro:property name="joint_2_max_position" value="${90.0 *pi/180.0}"/>
-  <xacro:property name="joint_3_max_position" value="${170.0 *pi/180.0}"/>
-  <xacro:property name="joint_4_max_position" value="${130.0 *pi/180.0}"/>
-  <xacro:property name="joint_5_max_position" value="${250.0 *pi/180.0}"/>
-  <xacro:property name="joint_6_max_position" value="${160.0 *pi/180.0}"/>
-  <xacro:property name="joint_7_max_position" value="${250.0 *pi/180.0}"/>
-  <!-- JOINTS VELOCITIE LIMITS-->
-  <!-- Real Values: [1, 1, 2, 2, 2, 2*pi, 2*pi] (rad/sec)-->
-  <xacro:property name="joint_1_max_velocity" value="1.85"/>
-  <xacro:property name="joint_2_max_velocity" value="1.85"/>
-  <xacro:property name="joint_3_max_velocity" value="1.85"/>
-  <xacro:property name="joint_4_max_velocity" value="1.85"/>
-  <xacro:property name="joint_5_max_velocity" value="1.85"/>
-  <xacro:property name="joint_6_max_velocity" value="${1.8*pi}"/>
-  <xacro:property name="joint_7_max_velocity" value="${1.8*pi}"/>
-  <!-- JOINT DYNAMICS DAMPING + FRICTION-->
-  <!-- >> !! Not Real Values !! << -->
-  <!-- DAMPING -->
-  <xacro:property name="joint_1_damping" value="0.8"/>
-  <xacro:property name="joint_2_damping" value="0.8"/>
-  <xacro:property name="joint_3_damping" value="0.8"/>
-  <xacro:property name="joint_4_damping" value="0.8"/>
-  <xacro:property name="joint_5_damping" value="0.8"/>
-  <xacro:property name="joint_6_damping" value="0.8"/>
-  <xacro:property name="joint_7_damping" value="0.8"/>
-  <xacro:property name="joint_finger_damping" value="0.8"/>
-  <!-- FRICTION -->
-  <xacro:property name="joint_1_friction" value="0.1"/>
-  <xacro:property name="joint_2_friction" value="0.1"/>
-  <xacro:property name="joint_3_friction" value="0.1"/>
-  <xacro:property name="joint_4_friction" value="0.1"/>
-  <xacro:property name="joint_5_friction" value="0.1"/>
-  <xacro:property name="joint_6_friction" value="0.1"/>
-  <xacro:property name="joint_7_friction" value="0.1"/>
-  <xacro:property name="joint_finger_friction" value="0.1"/>
+  <!-- PA10 Properties -->
+  <xacro:include filename="$(find pa10_description)/urdf/pa10properties.xacro"/>
   <!-- Import all Gazebo-customization elements, including Gazebo colors -->
   <xacro:include filename="$(find pa10_description)/urdf/pa10csl.gazebo.urdf.xacro" />
@@ -70,31 +23,8 @@
   <!-- Import Transmitions -->
   <xacro:include filename="$(find pa10_description)/urdf/arm.transmission.xacro"/>
+  <!-- Import sensors -->
+  <xacro:include filename="$(find pa10_description)/urdf/sensors.urdf.xacro"/>
   <!-- LINKS -->
   <link name="world"/>
-  <xacro:if value="${enable_camera_}">
-    <link name="kinect2_rgb_optical_frame">
-      <visual>
-        <origin rpy="${pi} ${-pi/2.0} ${-pi/2.0}" xyz="0 0 0"/>
-        <geometry>
-          <mesh filename="package://pa10_description/sensors_3D_models/kinect.dae" scale="1 1 1"/>
-        </geometry>
-        <material name="">
-          <color rgba="0.0 0.0 0.0 1.0"/>
-        </material>
-      </visual>
-      <collision>
-        <origin rpy="${pi} ${-pi/2.0} ${-pi/2.0}" xyz="0 0 0"/>
-        <geometry>
-          <mesh filename="package://pa10_description/sensors_3D_models/kinect.dae" scale="1 1 1"/>
-        </geometry>
-      </collision>
-      <inertial>
-        <origin rpy="0 0 0" xyz="0 0 1"/>
-        <mass value="0.5"/>
-        <inertia ixx="0.001" ixy="0.0" ixz="0.0" iyy="0.001" iyz="0.0" izz="0.001"/>
-      </inertial>
-    </link>
-    <link name="kinect2_ir_optical_frame"/>
-  </xacro:if>
   <link name="base_link">
     <visual>
@@ -113,14 +43,71 @@
     </collision>
     <inertial>
-      <origin rpy="0 0 3.14" xyz="0 0 0.1"/>
+      <origin rpy="0 0 3.14" xyz="0 0 0.0"/>
+      <mass value="${mass_shoulder}"/>
+      <!-- <xacro:inertia_box height="${inertia_height_shoulder}" mass="${mass_shoulder}"/> -->
+      <!-- <xacro:inertia_cylinder height="0.2"  radius = "0.1" mass="0.5"/> -->
+      <inertia ixx="0.1" ixy="0.0" ixz="0.0" iyy="0.1" iyz="0.0" izz="0.1"/>
+    </inertial>
+  </link>
+  <link name="link_shoulder_1">
+    <visual>
+      <origin rpy="0 0 0" xyz="0 0 0.117"/>
+      <geometry>
+        <mesh filename="package://pa10_description/pa10_stl/S2.stl" scale="1 1 1"/>
+      </geometry>
+      <material name="">
+        <color rgba="0.88 0.88 0.88 1.0"/>
+      </material>
+    </visual>
+    <collision>
+      <origin rpy="0 0 0" xyz="0 0 0.117"/>
+      <geometry>
+        <mesh filename="package://pa10_description/pa10_stl_collision/S2_collision.stl" scale="1 1 1"/>
+      </geometry>
+    </collision>
+    <inertial>
+      <!-- <origin rpy="0 0 0" xyz="0 0 0.117"/> -->
+      <mass value="${mass_shoulder}"/>
+      <!-- <xacro:inertia_cylinder height="0.12"  radius = "0.08" mass="0.5"/> -->
+      <!-- <xacro:inertia_box height="${inertia_height_shoulder}" mass="${mass_shoulder}"/> -->
+      <inertia ixx="0.1" ixy="0.0" ixz="0.0" iyy="0.1" iyz="0.0" izz="0.1"/>
+    </inertial>
+  </link>
+  <link name="link_shoulder_2">
+    <visual>
+      <origin rpy="-1.57079 0 3.14159" xyz="0 0 0"/>
+      <geometry>
+        <mesh filename="package://pa10_description/pa10_stl/S3.stl" scale="1 1 1"/>
+      </geometry>
+      <material name="pa10_blue">
+      </material>
+    </visual>
+    <collision>
+      <origin rpy="-1.57079 0 3.14159" xyz="0 0 0"/>
+      <geometry>
+        <mesh filename="package://pa10_description/pa10_stl_collision/S3_collision.stl" scale="1 1 1"/>
+      </geometry>
+    </collision>
+    <inertial>
+      <origin rpy="-1.57079 0 3.14159" xyz="0 -0.0 0.0"/>
+      <mass value="${mass_shoulder}"/>
+      <!-- <xacro:inertia_cylinder height="0.18"  radius = "0.05" mass="0.5" axis="0"/> -->
+      <!-- <xacro:inertia_box height="${inertia_height_shoulder}" mass="${mass_shoulder}"/> -->
+      <inertia ixx="0.1" ixy="0.0" ixz="0.0" iyy="0.1" iyz="0.0" izz="0.1"/>
+    </inertial>
+  </link>
+  <link name="link_shoulder_to_elbow">
+    <inertial>
+      <origin rpy="0 0 0" xyz="0 0 0.0"/>
       <mass value="0.5"/>
-      <xacro:inertia_cylinder height="0.2"  radius = "0.1" mass="0.5"/>
-    </inertial>
-  </link>
-  <link name="link_shoulder_1">
-    <visual>
-      <origin rpy="0 0 0" xyz="0 0 0.117"/>
-      <geometry>
-        <mesh filename="package://pa10_description/pa10_stl/S2.stl" scale="1 1 1"/>
+      <!-- <xacro:inertia_box height="${inertia_height}" mass="${mass_shoulder}"/> -->
+      <inertia ixx="0.1" ixy="0.0" ixz="0.0" iyy="0.1" iyz="0.0" izz="0.1"/>
+    </inertial>
+  </link>
+  <link name="link_elbow_1">
+    <visual>
+      <origin rpy="0 0 0" xyz="0 0.0 0.133"/>
+      <geometry>
+        <mesh filename="package://pa10_description/pa10_stl/E1.stl" scale="1 1 1"/>
       </geometry>
       <material name="">
@@ -129,20 +116,22 @@
     </visual>
     <collision>
-      <origin rpy="0 0 0" xyz="0 0 0.117"/>
-      <geometry>
-        <mesh filename="package://pa10_description/pa10_stl_collision/S2_collision.stl" scale="1 1 1"/>
-      </geometry>
-    </collision>
-    <inertial>
-      <origin rpy="0 0 0" xyz="0 0 0.117"/>
-      <mass value="0.5"/>
-      <xacro:inertia_cylinder height="0.12"  radius = "0.08" mass="0.5"/>
-    </inertial>
-  </link>
-  <link name="link_shoulder_2">
-    <visual>
-      <origin rpy="-1.57079 0 3.14159" xyz="0 0 0"/>
-      <geometry>
-        <mesh filename="package://pa10_description/pa10_stl/S3.stl" scale="1 1 1"/>
+      <origin rpy="0 0 0" xyz="0 0.0 0.133"/>
+      <geometry>
+        <mesh filename="package://pa10_description/pa10_stl_collision/E1_collision.stl" scale="1 1 1"/>
+      </geometry>
+    </collision>
+    <inertial>
+      <!-- <origin rpy="0 0 0" xyz="0 0.0 0.133"/> -->
+      <mass value="${mass_elbow}"/>
+      <!-- <xacro:inertia_cylinder height="0.12"  radius = "0.08" mass="0.5"/> -->
+      <!-- <xacro:inertia_box height="${inertia_height_elbow}" mass="${mass_elbow}"/> -->
+      <inertia ixx="0.1" ixy="0.0" ixz="0.0" iyy="0.1" iyz="0.0" izz="0.1"/>
+    </inertial>
+  </link>
+  <link name="link_elbow_2">
+    <visual>
+      <origin rpy="1.57079 0 0" xyz="0 0.003 0"/>
+      <geometry>
+        <mesh filename="package://pa10_description/pa10_stl/E2.stl" scale="1 1 1"/>
       </geometry>
       <material name="pa10_blue">
@@ -150,27 +139,22 @@
     </visual>
     <collision>
-      <origin rpy="-1.57079 0 3.14159" xyz="0 0 0"/>
-      <geometry>
-        <mesh filename="package://pa10_description/pa10_stl_collision/S3_collision.stl" scale="1 1 1"/>
-      </geometry>
-    </collision>
-    <inertial>
-      <origin rpy="-1.57079 0 3.14159" xyz="0 -0.22 0.0"/>
-      <mass value="0.5"/>
-      <xacro:inertia_cylinder height="0.18"  radius = "0.05" mass="0.5" axis="0"/>
-    </inertial>
-  </link>
-  <link name="link_shoulder_to_elbow">
-    <inertial>
-      <origin rpy="0 0 0" xyz="0 0 0.22"/>
-      <mass value="0.5"/>
-      <inertia ixx="0.001" ixy="0.0" ixz="0.0" iyy="0.001" iyz="0.0" izz="0.001"/>
-    </inertial>
-  </link>
-  <link name="link_elbow_1">
-    <visual>
-      <origin rpy="0 0 0" xyz="0 0.0 0.133"/>
-      <geometry>
-        <mesh filename="package://pa10_description/pa10_stl/E1.stl" scale="1 1 1"/>
+      <origin rpy="1.57079 0 0" xyz="0 0.003 0"/>
+      <geometry>
+        <mesh filename="package://pa10_description/pa10_stl_collision/E2_collision.stl" scale="1 1 1"/>
+      </geometry>
+    </collision>
+    <inertial>
+      <origin rpy="1.57079 0 0" xyz="0 -0.0 0"/>
+      <mass value="${mass_elbow}"/>
+      <!-- <xacro:inertia_cylinder height="0.15"  radius = "0.05" mass="0.5" axis="0"/> -->
+      <!-- <xacro:inertia_box height="${inertia_height_elbow}" mass="${mass_elbow}"/> -->
+      <inertia ixx="0.1" ixy="0.0" ixz="0.0" iyy="0.1" iyz="0.0" izz="0.1"/>
+    </inertial>
+  </link>
+  <link name="link_wrist_1">
+    <visual>
+      <origin rpy="0 0 0" xyz="0 0 0.195"/>
+      <geometry>
+        <mesh filename="package://pa10_description/pa10_stl/W1.stl" scale="1 1 1"/>
       </geometry>
       <material name="">
@@ -179,20 +163,22 @@
     </visual>
     <collision>
-      <origin rpy="0 0 0" xyz="0 0.0 0.133"/>
-      <geometry>
-        <mesh filename="package://pa10_description/pa10_stl_collision/E1_collision.stl" scale="1 1 1"/>
-      </geometry>
-    </collision>
-    <inertial>
-      <origin rpy="0 0 0" xyz="0 0.0 0.133"/>
-      <mass value="0.5"/>
-      <xacro:inertia_cylinder height="0.12"  radius = "0.08" mass="0.5"/>
-    </inertial>
-  </link>
-  <link name="link_elbow_2">
-    <visual>
-      <origin rpy="1.57079 0 0" xyz="0 0.003 0"/>
-      <geometry>
-        <mesh filename="package://pa10_description/pa10_stl/E2.stl" scale="1 1 1"/>
+      <origin rpy="0 0 0" xyz="0 0 0.195"/>
+      <geometry>
+        <mesh filename="package://pa10_description/pa10_stl_collision/W1_collision.stl" scale="1 1 1"/>
+      </geometry>
+    </collision>
+    <inertial>
+      <!-- <origin rpy="0 0 0" xyz="0 0 0.195"/> -->
+      <mass value="${mass_wrist}"/>
+      <!-- <xacro:inertia_cylinder height="0.15"  radius = "0.08" mass="0.5"/> -->
+      <!-- <xacro:inertia_box height="${inertia_height_wrist}" mass="${mass_wrist}"/> -->
+      <inertia ixx="0.1" ixy="0.0" ixz="0.0" iyy="0.1" iyz="0.0" izz="0.1"/>
+    </inertial>
+  </link>
+  <link name="link_wrist_2">
+    <visual>
+      <origin rpy="1.57079 0 0" xyz="0 0 0"/>
+      <geometry>
+        <mesh filename="package://pa10_description/pa10_stl/W2.stl" scale="1 1 1"/>
       </geometry>
       <material name="pa10_blue">
@@ -200,64 +186,31 @@
     </visual>
     <collision>
-      <origin rpy="1.57079 0 0" xyz="0 0.003 0"/>
-      <geometry>
-        <mesh filename="package://pa10_description/pa10_stl_collision/E2_collision.stl" scale="1 1 1"/>
-      </geometry>
-    </collision>
-    <inertial>
-      <origin rpy="1.57079 0 0" xyz="0 -0.15 0"/>
-      <mass value="0.5"/>
-      <xacro:inertia_cylinder height="0.15"  radius = "0.05" mass="0.5" axis="0"/>
-    </inertial>
-  </link>
-  <link name="link_wrist_1">
-    <visual>
-      <origin rpy="0 0 0" xyz="0 0 0.195"/>
-      <geometry>
-        <mesh filename="package://pa10_description/pa10_stl/W1.stl" scale="1 1 1"/>
-      </geometry>
-      <material name="">
-        <color rgba="0.88 0.88 0.88 1.0"/>
-      </material>
-    </visual>
-    <collision>
-      <origin rpy="0 0 0" xyz="0 0 0.195"/>
-      <geometry>
-        <mesh filename="package://pa10_description/pa10_stl_collision/W1_collision.stl" scale="1 1 1"/>
-      </geometry>
-    </collision>
-    <inertial>
-      <origin rpy="0 0 0" xyz="0 0 0.195"/>
-      <mass value="0.5"/>
-      <xacro:inertia_cylinder height="0.15"  radius = "0.08" mass="0.5"/>
-    </inertial>
-  </link>
-  <link name="link_wrist_2">
-    <visual>
       <origin rpy="1.57079 0 0" xyz="0 0 0"/>
       <geometry>
-        <mesh filename="package://pa10_description/pa10_stl/W2.stl" scale="1 1 1"/>
-      </geometry>
-      <material name="pa10_blue">
-      </material>
-    </visual>
-    <collision>
+        <mesh filename="package://pa10_description/pa10_stl_collision/W2_collision.stl" scale="1 1 1"/>
+      </geometry>
+    </collision>
+    <inertial>
       <origin rpy="1.57079 0 0" xyz="0 0 0"/>
-      <geometry>
-        <mesh filename="package://pa10_description/pa10_stl_collision/W2_collision.stl" scale="1 1 1"/>
-      </geometry>
-    </collision>
-    <inertial>
-      <origin rpy="1.57079 0 0" xyz="0 0 0"/>
-      <mass value="0.5"/>
-      <xacro:inertia_cylinder height="0.05"  radius = "0.08" mass="0.5" axis="1"/>
-    </inertial>
-  </link>
-  <link name="link_wrist_3"/>
+      <mass value="${mass_wrist}"/>
+      <!-- <xacro:inertia_cylinder height="0.05"  radius = "0.08" mass="0.5" axis="1"/> -->
+      <!-- <xacro:inertia_box height="${inertia_height_wrist}" mass="${mass_wrist}"/> -->
+      <inertia ixx="0.1" ixy="0.0" ixz="0.0" iyy="0.1" iyz="0.0" izz="0.1"/>
+    </inertial>
+  </link>
+  <link name="link_wrist_3">
+    <inertial>
+      <origin rpy="0 0 0" xyz="0 0 0"/>
+      <mass value="0.01"/>
+      <inertia ixx="0.01" ixy="0.0" ixz="0.0" iyy="0.01" iyz="0.0" izz="0.01"/>
+      <!-- <xacro:inertia_box height="${inertia_height}" mass="${mass_wrist}"/> -->
+    </inertial>
+  </link>
   <link name="link_ee_tool">
     <inertial>
       <origin rpy="0 0 0" xyz="0 0 0"/>
-      <mass value="0.1"/>
-      <inertia ixx="0.001" ixy="0.0" ixz="0.0" iyy="0.001" iyz="0.0" izz="0.001"/>
+      <mass value="0.01"/>
+      <inertia ixx="0.01" ixy="0.0" ixz="0.0" iyy="0.01" iyz="0.0" izz="0.01"/>
+      <!-- <xacro:inertia_box height="${inertia_height}" mass="${mass_2}"/> -->
     </inertial>
   </link>
@@ -280,7 +233,9 @@
     </collision>
     <inertial>
-      <origin rpy="0 0 0" xyz="0 0 -0.045"/>
-      <mass value="0.2"/>
-      <xacro:inertia_cylinder height="0.05"  radius = "0.03" mass="0.2"/>
+      <!-- <origin rpy="0 0 0" xyz="0 0 -0.045"/> -->
+      <mass value="${mass_gripper}"/>
+      <!-- <xacro:inertia_cylinder height="0.05"  radius = "0.03" mass="0.5"/> -->
+      <!-- <xacro:inertia_box height="${inertia_height_gripper}" mass="${mass_gripper}"/> -->
+      <inertia ixx="0.1" ixy="0.0" ixz="0.0" iyy="0.1" iyz="0.0" izz="0.1"/>
     </inertial>
   </link>
@@ -302,5 +257,7 @@
     </collision>
     <inertial>
-      <mass value="0.1"/>
+      <mass value="${mass_gripper}"/>
+      <!-- <inertia ixx="0.01" ixy="0.0" ixz="0.0" iyy="0.01" iyz="0.0" izz="0.01"/> -->
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
File: pa10_description/urdf/pa10csl.gazebo.urdf.xacro (robot description, xacro)
@@ -32,4 +32,17 @@
     </xacro:unless>
   </xacro:macro>
+  <!-- Inertial of Box -->
+  <xacro:macro name="inertia_box" params="mass height:=0.05 width:=0.0 depth:=0.0">
+    <xacro:if value="${width == 0.0}">
+      <xacro:property name="width" value="${height}"/>
+    </xacro:if>
+    <xacro:if value="${depth == 0.0}">
+      <xacro:property name="depth" value="${height}"/>
+    </xacro:if>
+    <xacro:property name="Iw" value="${(1.0/12.0)*mass*(height*height + depth*depth)}" />
+    <xacro:property name="Ih" value="${(1.0/12.0)*mass*(width*width + depth*depth)}" />
+    <xacro:property name="Id" value="${(1.0/12.0)*mass*(width*width + height*height)}" />
+    <inertia ixx="${Iw}" ixy="0" ixz="0" iyy="${Ih}" iyz="0" izz="${Id}" />
+  </xacro:macro>
   <!-- Gazebo Colors Material -->
   <xacro:macro name="gazebo_materials" params="prefix:='' color:='default'">
@@ -233,46 +246,3 @@
     </material>
   </gazebo>
-  <xacro:macro name="depth_sensor" params="link_name camera_name:='kinect' update_rate:=10">
-    <gazebo reference="${link_name}">
-      <sensor name="${link_name}_camera" type="depth">
-        <update_rate>${update_rate}</update_rate>
-        <camera>
-          <horizontal_fov>1.047198</horizontal_fov>
-          <image>
-            <width>640</width>
-            <height>480</height>
-            <format>R8G8B8</format>
-          </image>
-          <clip>
-            <near>0.05</near>
-            <far>3</far>
-          </clip>
-        </camera>
-        <plugin name="${link_name}_controller" filename="libgazebo_ros_openni_kinect.so">
-          <baseline>0.2</baseline>
-          <alwaysOn>true</alwaysOn>
-          <updateRate>1.0</updateRate>
-          <cameraName>${camera_name}_ir_${nsp}</cameraName>
-          <imageTopicName>${nsp}/${camera_name}/color/image_raw</imageTopicName>
-          <cameraInfoTopicName>${nsp}/${camera_name}/color/camera_info</cameraInfoTopicName>
-          <depthImageTopicName>${nsp}/${camera_name}/depth/image_raw</depthImageTopicName>
-          <depthImageInfoTopicName>${nsp}/${camera_name}/depth/camera_info</depthImageInfoTopicName>
-          <pointCloudTopicName>${nsp}/${camera_name}/depth/points</pointCloudTopicName>
-          <frameName>${camera_name}_${nsp}</frameName>
-          <pointCloudCutoff>0.5</pointCloudCutoff>
-          <pointCloudCutoffMax>3.0</pointCloudCutoffMax>
-          <distortionK1>0.00000001</distortionK1>
-          <distortionK2>0.00000001</distortionK2>
-          <distortionK3>0.00000001</distortionK3>
-          <distortionT1>0.00000001</distortionT1>
-          <distortionT2>0.00000001</distortionT2>
-          <CxPrime>0</CxPrime>
-          <Cx>0</Cx>
-          <Cy>0</Cy>
-          <focalLength>0</focalLength>
-          <hackBaseline>0</hackBaseline>
-        </plugin>
-      </sensor>
-    </gazebo>
-  </xacro:macro>
 </robot>
